Commit message: Change the joint limit from pi to 2pi in ur5.urdf.xacro
Change the joint limit and test the Cartesian motion separately. left_ and right_ worked well but arms_ didn't

File: dual_arm_robot_description/urdf/ur5.urdf.xacro (robot description, xacro)
@@ -97,5 +97,5 @@
       </xacro:unless>
       <xacro:if value="${joint_limited}">
-        <limit lower="${-pi}" upper="${pi}" effort="150.0" velocity="3.15"/>
+        <limit lower="${-2*pi}" upper="${2*pi}" effort="150.0" velocity="3.15"/>
       </xacro:if>
       <dynamics damping="0.0" friction="0.0"/>
@@ -128,5 +128,5 @@
       </xacro:unless>
       <xacro:if value="${joint_limited}">
-        <limit lower="${-pi}" upper="${pi}" effort="150.0" velocity="3.15"/>
+        <limit lower="${-2.0*pi}" upper="${2.*pi}" effort="150.0" velocity="3.15"/>
       </xacro:if>
       <dynamics damping="0.0" friction="0.0"/>
@@ -159,5 +159,5 @@
       </xacro:unless>
       <xacro:if value="${joint_limited}">
-        <limit lower="${-pi}" upper="${pi}" effort="150.0" velocity="3.15"/>
+        <limit lower="${-2*pi}" upper="${2*pi}" effort="150.0" velocity="3.15"/>
       </xacro:if>
       <dynamics damping="0.0" friction="0.0"/>
@@ -190,5 +190,5 @@
       </xacro:unless>
       <xacro:if value="${joint_limited}">
-        <limit lower="${-pi}" upper="${pi}" effort="28.0" velocity="3.2"/>
+        <limit lower="${-2*pi}" upper="${2*pi}" effort="28.0" velocity="3.2"/>
       </xacro:if>
       <dynamics damping="0.0" friction="0.0"/>
@@ -221,5 +221,5 @@
       </xacro:unless>
       <xacro:if value="${joint_limited}">
-        <limit lower="${-pi}" upper="${pi}" effort="28.0" velocity="3.2"/>
+        <limit lower="${-2*pi}" upper="${2*pi}" effort="28.0" velocity="3.2"/>
       </xacro:if>
       <dynamics damping="0.0" friction="0.0"/>
@@ -252,5 +252,5 @@
       </xacro:unless>
       <xacro:if value="${joint_limited}">
-        <limit lower="${-pi}" upper="${pi}" effort="28.0" velocity="3.2"/>
+        <limit lower="${-2*pi}" upper="${2*pi}" effort="28.0" velocity="3.2"/>
       </xacro:if>
       <dynamics damping="0.0" friction="0.0"/>

Commit message: Rewrite the format of logdata

File: dual_arm_robot_description/urdf/ur5.urdf.xacro (robot description, xacro)
@@ -94,5 +94,5 @@
       <axis xyz="0 0 1" />
       <xacro:unless value="${joint_limited}">
-        <limit lower="${-2.0 * pi}" upper="${2.0 * pi}" effort="150.0" velocity="3.15"/>
+        <limit lower="${-pi}" upper="${pi}" effort="150.0" velocity="3.15"/>
       </xacro:unless>
       <xacro:if value="${joint_limited}">
@@ -125,5 +125,5 @@
       <axis xyz="0 1 0" />
       <xacro:unless value="${joint_limited}">
-        <limit lower="${-2.0 * pi}" upper="${2.0 * pi}" effort="150.0" velocity="3.15"/>
+        <limit lower="${-pi}" upper="${pi}" effort="150.0" velocity="3.15"/>
       </xacro:unless>
       <xacro:if value="${joint_limited}">
@@ -156,5 +156,5 @@
       <axis xyz="0 1 0" />
       <xacro:unless value="${joint_limited}">
-        <limit lower="${-2.0 * pi}" upper="${2.0 * pi}" effort="150.0" velocity="3.15"/>
+        <limit lower="${-pi}" upper="${pi}" effort="150.0" velocity="3.15"/>
       </xacro:unless>
       <xacro:if value="${joint_limited}">
@@ -187,5 +187,5 @@
       <axis xyz="0 1 0" />
       <xacro:unless value="${joint_limited}">
-        <limit lower="${-2.0 * pi}" upper="${2.0 * pi}" effort="28.0" velocity="3.2"/>
+        <limit lower="${-pi}" upper="${pi}" effort="28.0" velocity="3.2"/>
       </xacro:unless>
       <xacro:if value="${joint_limited}">
@@ -218,5 +218,5 @@
       <axis xyz="0 0 1" />
       <xacro:unless value="${joint_limited}">
-        <limit lower="${-2.0 * pi}" upper="${2.0 * pi}" effort="28.0" velocity="3.2"/>
+        <limit lower="${-pi}" upper="${pi}" effort="28.0" velocity="3.2"/>
       </xacro:unless>
       <xacro:if value="${joint_limited}">
@@ -252,5 +252,5 @@
       </xacro:unless>
       <xacro:if value="${joint_limited}">
-        <limit lower="${-pi}" upper="${pi}" effort="28.0" velocity="3.2"/>
+        <limit lower="${-2*pi}" upper="${2*pi}" effort="28.0" velocity="3.2"/>
       </xacro:if>
       <dynamics damping="0.0" friction="0.0"/>

Commit message: Change the iksolver from KDL to urkinematicsplugin

File: dual_arm_robot_description/urdf/ur5.urdf.xacro (robot description, xacro)
@@ -94,8 +94,8 @@
       <axis xyz="0 0 1" />
       <xacro:unless value="${joint_limited}">
-        <limit lower="${-pi}" upper="${pi}" effort="150.0" velocity="3.15"/>
-      </xacro:unless>
-      <xacro:if value="${joint_limited}">
-        <limit lower="${-pi}" upper="${pi}" effort="150.0" velocity="3.15"/>
+        <limit lower="${-pi}" upper="${pi}" effort="150.0" velocity="2"/>
+      </xacro:unless>
+      <xacro:if value="${joint_limited}">
+        <limit lower="${-pi}" upper="${pi}" effort="150.0" velocity="2"/>
       </xacro:if>
       <dynamics damping="0.0" friction="0.0"/>
@@ -125,8 +125,8 @@
       <axis xyz="0 1 0" />
       <xacro:unless value="${joint_limited}">
-        <limit lower="${-pi}" upper="${pi}" effort="150.0" velocity="3.15"/>
-      </xacro:unless>
-      <xacro:if value="${joint_limited}">
-        <limit lower="${-2.0*pi}" upper="${2.*pi}" effort="150.0" velocity="3.15"/>
+        <limit lower="${-pi}" upper="${pi}" effort="150.0" velocity="2"/>
+      </xacro:unless>
+      <xacro:if value="${joint_limited}">
+        <limit lower="${-2.0*pi}" upper="${2.*pi}" effort="150.0" velocity="2"/>
       </xacro:if>
       <dynamics damping="0.0" friction="0.0"/>
@@ -156,8 +156,8 @@
       <axis xyz="0 1 0" />
       <xacro:unless value="${joint_limited}">
-        <limit lower="${-pi}" upper="${pi}" effort="150.0" velocity="3.15"/>
-      </xacro:unless>
-      <xacro:if value="${joint_limited}">
-        <limit lower="${-pi}" upper="${pi}" effort="150.0" velocity="3.15"/>
+        <limit lower="${-pi}" upper="${pi}" effort="150.0" velocity="2"/>
+      </xacro:unless>
+      <xacro:if value="${joint_limited}">
+        <limit lower="${-pi}" upper="${pi}" effort="150.0" velocity="2"/>
       </xacro:if>
       <dynamics damping="0.0" friction="0.0"/>
@@ -187,8 +187,8 @@
       <axis xyz="0 1 0" />
       <xacro:unless value="${joint_limited}">
-        <limit lower="${-pi}" upper="${pi}" effort="28.0" velocity="3.2"/>
-      </xacro:unless>
-      <xacro:if value="${joint_limited}">
-        <limit lower="${-pi}" upper="${pi}" effort="28.0" velocity="3.2"/>
+        <limit lower="${-pi}" upper="${pi}" effort="28.0" velocity="2"/>
+      </xacro:unless>
+      <xacro:if value="${joint_limited}">
+        <limit lower="${-pi}" upper="${pi}" effort="28.0" velocity="2"/>
       </xacro:if>
       <dynamics damping="0.0" friction="0.0"/>
@@ -218,8 +218,8 @@
       <axis xyz="0 0 1" />
       <xacro:unless value="${joint_limited}">
-        <limit lower="${-pi}" upper="${pi}" effort="28.0" velocity="3.2"/>
-      </xacro:unless>
-      <xacro:if value="${joint_limited}">
-        <limit lower="${-pi}" upper="${pi}" effort="28.0" velocity="3.2"/>
+        <limit lower="${-pi}" upper="${pi}" effort="28.0" velocity="2"/>
+      </xacro:unless>
+      <xacro:if value="${joint_limited}">
+        <limit lower="${-2*pi}" upper="${2*pi}" effort="28.0" velocity="2"/>
       </xacro:if>
       <dynamics damping="0.0" friction="0.0"/>
@@ -249,8 +249,8 @@
       <axis xyz="0 1 0" />
       <xacro:unless value="${joint_limited}">
-        <limit lower="${-pi}" upper="${pi}" effort="28.0" velocity="3.2"/>
-      </xacro:unless>
-      <xacro:if value="${joint_limited}">
-        <limit lower="${-2*pi}" upper="${2*pi}" effort="28.0" velocity="3.2"/>
+        <limit lower="${-pi}" upper="${pi}" effort="28.0" velocity="2"/>
+      </xacro:unless>
+      <xacro:if value="${joint_limited}">
+        <limit lower="${-2*pi}" upper="${2*pi}" effort="28.0" velocity="2"/>
       </xacro:if>
       <dynamics damping="0.0" friction="0.0"/>

Commit message: Transfer to the new pc

File: dual_arm_robot_description/urdf/ur5.urdf.xacro (robot description, xacro)
@@ -128,5 +128,5 @@
       </xacro:unless>
       <xacro:if value="${joint_limited}">
-        <limit lower="${-2.0*pi}" upper="${2.*pi}" effort="150.0" velocity="2"/>
+        <limit lower="${-pi}" upper="${pi}" effort="150.0" velocity="2"/>
       </xacro:if>
       <dynamics damping="0.0" friction="0.0"/>
@@ -277,5 +277,6 @@
       <parent link="${prefix}wrist_3_link" />
       <child link = "${prefix}ee_link" />
-      <origin xyz="0.0 ${ur5_wrist_3_length} 0.0" rpy="${pi/2} ${pi} ${-pi}" />
+      <!--origin xyz="0.0 ${ur5_wrist_3_length} 0.0" rpy="${pi/2} ${pi} ${-pi}" /-->
+      <origin xyz="0.0 ${ur5_wrist_3_length} 0.0" rpy="0.0 0.0 ${pi/2.0}" />
     </joint>
     <link name="${prefix}ee_link">
@@ -301,5 +302,4 @@
     </joint>
     <!-- Frame coincident with all-zeros TCP on UR controller -->
-    <!--
     <link name="${prefix}tool0"/>
     <joint name="${prefix}wrist_3_link-tool0_fixed_joint" type="fixed">
@@ -308,5 +308,4 @@
       <child link="${prefix}tool0"/>
     </joint>
-    -->
   </xacro:macro>
 </robot>
