Commit message: Change 'ur10' to 'right'
Change all the parameters involved with 'ur10' to 'right'

File: dual_arm_robot_description/urdf/dual_arm_robot.urdf.xacro (robot description, xacro)
@@ -4,7 +4,7 @@
   <xacro:property name="pi" value="3.1415926535897931"/>
   <xacro:arg name="prefix_ur5" default="ur5_"/>
-  <xacro:arg name="prefix_ur10" default="right_"/>
+  <xacro:arg name="prefix_right" default="right_"/>
   <xacro:arg name="limited_ur5" default="true"/>
-  <xacro:arg name="limited_ur10" default="true"/>
+  <xacro:arg name="limited_right" default="true"/>
   <!-- common stuff -->
   <xacro:include filename="$(find ur_description)/urdf/common.gazebo.xacro"/>
@@ -12,5 +12,5 @@
   <xacro:include filename="$(find dual_arm_robot_description)/urdf/ur5.urdf.xacro"/> <!-- file has been edited because of same variable names in ur5 and ur10 -->
   <!-- ur10 -->
-  <xacro:include filename="$(find dual_arm_robot_description)/urdf/ur5.urdf.xacro"/> <!-- original file has been edited because of same variable names in ur5 and ur10 -->
+  <xacro:include filename="$(find dual_arm_robot_description)/urdf/ur5_right.urdf.xacro"/> <!-- original file has been edited because of same variable names in ur5 and ur10 -->
   <!-- endeffector -->
   <xacro:include filename="$(find dual_arm_robot_description)/urdf/endeffector.urdf.xacro"/>
@@ -48,21 +48,21 @@
 -->
   <!-- place ur10 arm -->
-  <xacro:ur10_robot prefix="$(arg prefix_ur10)" joint_limited="$(arg limited_ur10)"/>
-  <joint name="$(arg prefix_ur10)platform_mount" type="fixed">
-    <parent link="$(arg prefix_ur10)table_platform"/>
-    <child link ="$(arg prefix_ur10)base_link"/>
+  <xacro:right_robot prefix="$(arg prefix_right)" joint_limited="$(arg limited_right)"/>
+  <joint name="$(arg prefix_right)platform_mount" type="fixed">
+    <parent link="$(arg prefix_right)table_platform"/>
+    <child link ="$(arg prefix_right)base_link"/>
     <origin xyz="0.1341 -0.3049 0.0155" rpy="0 0 ${pi/2}" />
   </joint>
   <!-- place ur10 endeffector -->
-  <xacro:endeffector prefix="$(arg prefix_ur10)"/>
-  <joint name="$(arg prefix_ur10)ee_mount" type="fixed">
-    <parent link="$(arg prefix_ur10)ee_link" />
-    <child link = "$(arg prefix_ur10)ee_frame" />
+  <xacro:endeffector prefix="$(arg prefix_right)"/>
+  <joint name="$(arg prefix_right)ee_mount" type="fixed">
+    <parent link="$(arg prefix_right)ee_link" />
+    <child link = "$(arg prefix_right)ee_frame" />
     <origin xyz="0.0 0.0 0.0" rpy="${pi/2.0} 0.0 ${pi/2.0}" />
   </joint>
 <!--
-  <joint name="$(arg prefix_ur10)ee_mount" type="fixed">
-    <parent link="$(arg prefix_ur10)tool0"/>
-    <child link ="$(arg prefix_ur10)ee_frame"/>
+  <joint name="$(arg prefix_right)ee_mount" type="fixed">
+    <parent link="$(arg prefix_right)tool0"/>
+    <child link ="$(arg prefix_right)ee_frame"/>
     <origin xyz="0 0 0" rpy="0 0 ${pi}" />
   </joint>

File: dual_arm_robot_description/urdf/table.urdf.xacro (robot description, xacro)
@@ -142,8 +142,8 @@
     <origin xyz="0 0 0"/>
   </joint>
-  <link name="$(arg prefix_ur10)table_platform">
+  <link name="$(arg prefix_right)table_platform">
     <visual>
       <geometry>
-        <mesh filename="package://dual_arm_robot_description/meshes/table/table_platform_ur10.stl"/>
+        <mesh filename="package://dual_arm_robot_description/meshes/table/table_platform_right.stl"/>
       </geometry>
     <material name="steel"/>
@@ -152,11 +152,11 @@
     <collision>
       <geometry>
-        <mesh filename="package://dual_arm_robot_description/meshes/table/table_platform_ur10.stl"/>
+        <mesh filename="package://dual_arm_robot_description/meshes/table/table_platform_right.stl"/>
       </geometry>
     </collision>
   </link>
-  <joint name="$(arg prefix_ur10)table_ground_to_platform" type="fixed">
+  <joint name="$(arg prefix_right)table_ground_to_platform" type="fixed">
     <parent link="table_ground"/>
-    <child link="$(arg prefix_ur10)table_platform"/>
+    <child link="$(arg prefix_right)table_platform"/>
     <origin xyz="1.076 0 0"/>
   </joint>

File: dual_arm_robot_description/urdf/ur5_right.urdf.xacro (robot description, xacro)
@@ -2,47 +2,62 @@
 <robot xmlns:xacro="http://www.ros.org/wiki/xacro">
 <!-- edited by Daniel Hoeltgen-->
-<!--
-  Author: Kelsey Hawkins
-  Contributers: Jimmy Da Silva, Ajit Krisshna N L, Muhammad Asif Rana
--->
   <xacro:include filename="$(find ur_description)/urdf/ur.transmission.xacro" />
   <xacro:include filename="$(find ur_description)/urdf/ur.gazebo.xacro" />
   <property name="pi" value="3.14159265" />
   <!-- Inertia parameters -->
-  <property name="right_base_mass" value="4.0" />  <!-- This mass might be incorrect -->
-  <property name="right_shoulder_mass" value="7.778" />
-  <property name="right_upper_arm_mass" value="12.93" />
-  <property name="right_forearm_mass" value="3.87" />
-  <property name="right_wrist_1_mass" value="1.96" />
-  <property name="right_wrist_2_mass" value="1.96" />
-  <property name="right_wrist_3_mass" value="0.202" />
-  <!-- These parameters are borrowed from the urcontrol.conf file
-       but are not verified for the correct permutation.
-       The permutation was guessed by looking at the UR5 parameters.
-       Serious use of these parameters needs further inspection. -->
-  <property name="right_shoulder_cog" value="0.00008 0.00244 -0.037" />
-  <property name="right_upper_arm_cog" value="0.00001 0.15061 0.38757" />
-  <property name="right_forearm_cog" value="-0.00012 0.06112 0.1984" />
-  <property name="right_wrist_1_cog" value="-0.00021 -0.00112 0.02269" />
-  <property name="right_wrist_2_cog" value="-0.00021 0.00112 0.002269" />
-  <property name="right_wrist_3_cog" value="0 -0.001156 -0.00149" />
+  <property name="ur5_base_mass" value="4.0" />  <!-- This mass might be incorrect -->
+  <property name="ur5_shoulder_mass" value="3.7000" />
+  <property name="ur5_upper_arm_mass" value="8.3930" />
+  <property name="ur5_forearm_mass" value="2.2750" />
+  <property name="ur5_wrist_1_mass" value="1.2190" />
+  <property name="ur5_wrist_2_mass" value="1.2190" />
+  <property name="ur5_wrist_3_mass" value="0.1879" />
+  <property name="ur5_shoulder_cog" value="0.0 0.00193 -0.02561" />
+  <property name="ur5_upper_arm_cog" value="0.0 -0.024201 0.2125" />
+  <property name="ur5_forearm_cog" value="0.0 0.0265 0.11993" />
+  <property name="ur5_wrist_1_cog" value="0.0 0.110949 0.01634" />
+  <property name="ur5_wrist_2_cog" value="0.0 0.0018 0.11099" />
+  <property name="ur5_wrist_3_cog" value="0.0 0.001159 0.0" />
   <!-- Kinematic model -->
   <!-- Properties from urcontrol.conf -->
-  <property name="right_d1" value="0.1273" />
-  <property name="right_a2" value="-0.612" />
-  <property name="right_a3" value="-0.5723" />
-  <property name="right_d4" value="0.163941" />
-  <property name="right_d5" value="0.1157" />
-  <property name="right_d6" value="0.0922" />
+  <!--
+    DH for UR5:
+    a = [0.00000, -0.42500, -0.39225,  0.00000,  0.00000,  0.0000]
+    d = [0.089159,  0.00000,  0.00000,  0.10915,  0.09465,  0.0823]
+    alpha = [ 1.570796327, 0, 0, 1.570796327, -1.570796327, 0 ]
+    q_home_offset = [0, -1.570796327, 0, -1.570796327, 0, 0]
+    joint_direction = [-1, -1, 1, 1, 1, 1]
+    mass = [3.7000, 8.3930, 2.2750, 1.2190, 1.2190, 0.1879]
+    center_of_mass = [ [0, -0.02561, 0.00193], [0.2125, 0, 0.11336], [0.11993, 0.0, 0.0265], [0, -0.0018, 0.01634], [0, 0.0018,0.01634], [0, 0, -0.001159] ]
+  -->
+  <property name="ur5_d1" value="0.089159" />
+  <property name="ur5_a2" value="-0.42500" />
+  <property name="ur5_a3" value="-0.39225" />
+  <property name="ur5_d4" value="0.10915" />
+  <property name="ur5_d5" value="0.09465" />
+  <property name="ur5_d6" value="0.0823" />
   <!-- Arbitrary offsets for shoulder/elbow joints -->
-  <property name="right_shoulder_offset" value="0.220941" />  <!-- measured from model -->
-  <property name="right_elbow_offset" value="-0.1719" /> <!-- measured from model -->
+  <property name="ur5_shoulder_offset" value="0.13585" />  <!-- measured from model -->
+  <property name="ur5_elbow_offset" value="-0.1197" /> <!-- measured from model -->
   <!-- link lengths used in model -->
-  <property name="right_shoulder_height" value="${right_d1}" />
-  <property name="right_upper_arm_length" value="${-right_a2}" />
-  <property name="right_forearm_length" value="${-right_a3}" />
-  <property name="right_wrist_1_length" value="${right_d4 - right_elbow_offset - right_shoulder_offset}" />
-  <property name="right_wrist_2_length" value="${right_d5}" />
-  <property name="right_wrist_3_length" value="${right_d6}" />
+  <property name="ur5_shoulder_height" value="${ur5_d1}" />
+  <property name="ur5_upper_arm_length" value="${-ur5_a2}" />
+  <property name="ur5_forearm_length" value="${-ur5_a3}" />
+  <property name="ur5_wrist_1_length" value="${ur5_d4 - ur5_elbow_offset - ur5_shoulder_offset}" />
+  <property name="ur5_wrist_2_length" value="${ur5_d5}" />
+  <property name="ur5_wrist_3_length" value="${ur5_d6}" />
+  <!--property name="ur5_shoulder_height" value="0.089159" /-->
+  <!--property name="ur5_shoulder_offset" value="0.13585" /-->  <!-- ur5_shoulder_offset - ur5_elbow_offset + ur5_wrist_1_length = 0.10915 -->
+  <!--property name="ur5_upper_arm_length" value="0.42500" /-->
+  <!--property name="ur5_elbow_offset" value="0.1197" /-->       <!-- CAD measured -->
+  <!--property name="ur5_forearm_length" value="0.39225" /-->
+  <!--property name="ur5_wrist_1_length" value="0.093" /-->     <!-- CAD measured -->
+  <!--property name="ur5_wrist_2_length" value="0.09465" /-->   <!-- In CAD this distance is 0.930, but in the spec it is 0.09465 -->
+  <!--property name="ur5_wrist_3_length" value="0.0823" /-->
+  <property name="ur5_shoulder_radius" value="0.060" />   <!-- manually measured -->
+  <property name="ur5_upper_arm_radius" value="0.054" />  <!-- manually measured -->
+  <property name="ur5_elbow_radius" value="0.060" />      <!-- manually measured -->
+  <property name="ur5_forearm_radius" value="0.040" />    <!-- manually measured -->
+  <property name="ur5_wrist_radius" value="0.045" />      <!-- manually measured -->
   <xacro:macro name="cylinder_inertial" params="radius length mass *origin">
     <inertial>
@@ -58,16 +73,16 @@
       <visual>
         <geometry>
-          <mesh filename="package://ur_description/meshes/ur10/visual/base.dae"/>
-        </geometry>
-        <material name="LightGrey">
-          <color rgba="0.7 0.7 0.7 1.0"/>
-        </material>
-      </visual>
-      <collision>
-        <geometry>
-          <mesh filename="package://ur_description/meshes/ur10/collision/base.stl"/>
-        </geometry>
-      </collision>
-      <xacro:cylinder_inertial radius="0.075" length="0.038" mass="${right_base_mass}">
+          <mesh filename="package://ur_description/meshes/ur5/visual/base.dae" />
+        </geometry>
+        <material name="LightGrey">
+          <color rgba="0.7 0.7 0.7 1.0"/>
+        </material>
+      </visual>
+      <collision>
+        <geometry>
+          <mesh filename="package://ur_description/meshes/ur5/collision/base.stl" />
+        </geometry>
+      </collision>
+      <xacro:cylinder_inertial radius="0.06" length="0.05" mass="${ur5_base_mass}">
         <origin xyz="0.0 0.0 0.0" rpy="0 0 0" />
       </xacro:cylinder_inertial>
@@ -76,11 +91,11 @@
       <parent link="${prefix}base_link" />
       <child link = "${prefix}shoulder_link" />
-      <origin xyz="0.0 0.0 ${right_shoulder_height}" rpy="0.0 0.0 0.0" />
+      <origin xyz="0.0 0.0 ${ur5_shoulder_height}" rpy="0.0 0.0 0.0" />
       <axis xyz="0 0 1" />
       <xacro:unless value="${joint_limited}">
-        <limit lower="${-2.0 * pi}" upper="${2.0 * pi}" effort="330.0" velocity="2.16"/>
-      </xacro:unless>
-      <xacro:if value="${joint_limited}">
-        <limit lower="${-pi}" upper="${pi}" effort="330.0" velocity="2.16"/>
+        <limit lower="${-2.0 * pi}" upper="${2.0 * pi}" effort="150.0" velocity="3.15"/>
+      </xacro:unless>
+      <xacro:if value="${joint_limited}">
+        <limit lower="${-pi}" upper="${pi}" effort="150.0" velocity="3.15"/>
       </xacro:if>
       <dynamics damping="0.0" friction="0.0"/>
@@ -89,16 +104,16 @@
       <visual>
         <geometry>
-          <mesh filename="package://ur_description/meshes/ur10/visual/shoulder.dae"/>
-        </geometry>
-        <material name="LightGrey">
-          <color rgba="0.7 0.7 0.7 1.0"/>
-        </material>
-      </visual>
-      <collision>
-        <geometry>
-          <mesh filename="package://ur_description/meshes/ur10/collision/shoulder.stl"/>
-        </geometry>
-      </collision>
-      <xacro:cylinder_inertial radius="0.075" length="0.178" mass="${right_shoulder_mass}">
+          <mesh filename="package://ur_description/meshes/ur5/visual/shoulder.dae" />
+        </geometry>
+        <material name="LightGrey">
+          <color rgba="0.7 0.7 0.7 1.0"/>
+        </material>
+      </visual>
+      <collision>
+        <geometry>
+          <mesh filename="package://ur_description/meshes/ur5/collision/shoulder.stl" />
+        </geometry>
+      </collision>
+      <xacro:cylinder_inertial radius="0.06" length="0.15" mass="${ur5_shoulder_mass}">
         <origin xyz="0.0 0.0 0.0" rpy="0 0 0" />
       </xacro:cylinder_inertial>
@@ -107,11 +122,11 @@
       <parent link="${prefix}shoulder_link" />
       <child link = "${prefix}upper_arm_link" />
-      <origin xyz="0.0 ${right_shoulder_offset} 0.0" rpy="0.0 ${pi / 2.0} 0.0" />
+      <origin xyz="0.0 ${ur5_shoulder_offset} 0.0" rpy="0.0 ${pi / 2.0} 0.0" />
       <axis xyz="0 1 0" />
       <xacro:unless value="${joint_limited}">
-        <limit lower="${-2.0 * pi}" upper="${2.0 * pi}" effort="330.0" velocity="2.16"/>
-      </xacro:unless>
-      <xacro:if value="${joint_limited}">
-        <limit lower="${-pi}" upper="${pi}" effort="330.0" velocity="2.16"/>
+        <limit lower="${-2.0 * pi}" upper="${2.0 * pi}" effort="150.0" velocity="3.15"/>
+      </xacro:unless>
+      <xacro:if value="${joint_limited}">
+        <limit lower="${-pi}" upper="${pi}" effort="150.0" velocity="3.15"/>
       </xacro:if>
       <dynamics damping="0.0" friction="0.0"/>
@@ -120,17 +135,17 @@
       <visual>
         <geometry>
-          <mesh filename="package://ur_description/meshes/ur10/visual/upperarm.dae"/>
-        </geometry>
-        <material name="LightGrey">
-          <color rgba="0.7 0.7 0.7 1.0"/>
-        </material>
-      </visual>
-      <collision>
-        <geometry>
-          <mesh filename="package://ur_description/meshes/ur10/collision/upperarm.stl"/>
-        </geometry>
-      </collision>
-      <xacro:cylinder_inertial radius="0.075" length="${-right_a2}" mass="${right_upper_arm_mass}">
-        <origin xyz="0.0 0.0 ${-right_a2/2.0}" rpy="0 0 0" />
+          <mesh filename="package://ur_description/meshes/ur5/visual/upperarm.dae" />
+        </geometry>
+        <material name="LightGrey">
+          <color rgba="0.7 0.7 0.7 1.0"/>
+        </material>
+      </visual>
+      <collision>
+        <geometry>
+          <mesh filename="package://ur_description/meshes/ur5/collision/upperarm.stl" />
+        </geometry>
+      </collision>
+      <xacro:cylinder_inertial radius="0.06" length="0.56" mass="${ur5_upper_arm_mass}">
+        <origin xyz="0.0 0.0 0.28" rpy="0 0 0" />
       </xacro:cylinder_inertial>
     </link>
@@ -138,5 +153,5 @@
       <parent link="${prefix}upper_arm_link" />
       <child link = "${prefix}forearm_link" />
-      <origin xyz="0.0 ${right_elbow_offset} ${right_upper_arm_length}" rpy="0.0 0.0 0.0" />
+      <origin xyz="0.0 ${ur5_elbow_offset} ${ur5_upper_arm_length}" rpy="0.0 0.0 0.0" />
       <axis xyz="0 1 0" />
       <xacro:unless value="${joint_limited}">
@@ -150,18 +165,18 @@
     <link name="${prefix}forearm_link">
       <visual>
-         <geometry>
-          <mesh filename="package://ur_description/meshes/ur10/visual/forearm.dae"/>
-        </geometry>
-        <material name="LightGrey">
-          <color rgba="0.7 0.7 0.7 1.0"/>
-        </material>
-      </visual>
-      <collision>
-        <geometry>
-          <mesh filename="package://ur_description/meshes/ur10/collision/forearm.stl"/>
-        </geometry>
-      </collision>
-      <xacro:cylinder_inertial radius="0.075" length="${-right_a3}" mass="${right_forearm_mass}">
-        <origin xyz="0.0 0.0 ${-right_a3/2.0}" rpy="0 0 0" />
+        <geometry>
+          <mesh filename="package://ur_description/meshes/ur5/visual/forearm.dae" />
+        </geometry>
+        <material name="LightGrey">
+          <color rgba="0.7 0.7 0.7 1.0"/>
+        </material>
+      </visual>
+      <collision>
+        <geometry>
+          <mesh filename="package://ur_description/meshes/ur5/collision/forearm.stl" />
+        </geometry>
+      </collision>
+      <xacro:cylinder_inertial radius="0.06" length="0.5" mass="${ur5_forearm_mass}">
+        <origin xyz="0.0 0.0 0.25" rpy="0 0 0" />
       </xacro:cylinder_inertial>
     </link>
@@ -169,11 +184,11 @@
       <parent link="${prefix}forearm_link" />
       <child link = "${prefix}wrist_1_link" />
-      <origin xyz="0.0 0.0 ${right_forearm_length}" rpy="0.0 ${pi / 2.0} 0.0" />
+      <origin xyz="0.0 0.0 ${ur5_forearm_length}" rpy="0.0 ${pi / 2.0} 0.0" />
       <axis xyz="0 1 0" />
       <xacro:unless value="${joint_limited}">
-        <limit lower="${-2.0 * pi}" upper="${2.0 * pi}" effort="54.0" velocity="3.2"/>
-      </xacro:unless>
-      <xacro:if value="${joint_limited}">
-        <limit lower="${-pi}" upper="${pi}" effort="54.0" velocity="3.2"/>
+        <limit lower="${-2.0 * pi}" upper="${2.0 * pi}" effort="28.0" velocity="3.2"/>
+      </xacro:unless>
+      <xacro:if value="${joint_limited}">
+        <limit lower="${-pi}" upper="${pi}" effort="28.0" velocity="3.2"/>
       </xacro:if>
       <dynamics damping="0.0" friction="0.0"/>
@@ -182,16 +197,16 @@
       <visual>
         <geometry>
-          <mesh filename="package://ur_description/meshes/ur10/visual/wrist1.dae"/>
-        </geometry>
-        <material name="LightGrey">
-          <color rgba="0.7 0.7 0.7 1.0"/>
-        </material>
-      </visual>
-      <collision>
-        <geometry>
-          <mesh filename="package://ur_description/meshes/ur10/collision/wrist1.stl"/>
-        </geometry>
-      </collision>
-      <xacro:cylinder_inertial radius="0.075" length="0.12" mass="${right_wrist_1_mass}">
+          <mesh filename="package://ur_description/meshes/ur5/visual/wrist1.dae" />
+        </geometry>
+        <material name="LightGrey">
+          <color rgba="0.7 0.7 0.7 1.0"/>
+        </material>
+      </visual>
+      <collision>
+        <geometry>
+          <mesh filename="package://ur_description/meshes/ur5/collision/wrist1.stl" />
+        </geometry>
+      </collision>
+      <xacro:cylinder_inertial radius="0.6" length="0.12" mass="${ur5_wrist_1_mass}">
         <origin xyz="0.0 0.0 0.0" rpy="0 0 0" />
       </xacro:cylinder_inertial>
@@ -200,11 +215,11 @@
       <parent link="${prefix}wrist_1_link" />
       <child link = "${prefix}wrist_2_link" />
-      <origin xyz="0.0 ${right_wrist_1_length} 0.0" rpy="0.0 0.0 0.0" />
+      <origin xyz="0.0 ${ur5_wrist_1_length} 0.0" rpy="0.0 0.0 0.0" />
       <axis xyz="0 0 1" />
       <xacro:unless value="${joint_limited}">
-        <limit lower="${-2.0 * pi}" upper="${2.0 * pi}" effort="54.0" velocity="3.2"/>
-      </xacro:unless>
-      <xacro:if value="${joint_limited}">
-        <limit lower="${-pi}" upper="${pi}" effort="54.0" velocity="3.2"/>
+        <limit lower="${-2.0 * pi}" upper="${2.0 * pi}" effort="28.0" velocity="3.2"/>
+      </xacro:unless>
+      <xacro:if value="${joint_limited}">
+        <limit lower="${-pi}" upper="${pi}" effort="28.0" velocity="3.2"/>
       </xacro:if>
       <dynamics damping="0.0" friction="0.0"/>
@@ -213,16 +228,16 @@
       <visual>
         <geometry>
-          <mesh filename="package://ur_description/meshes/ur10/visual/wrist2.dae"/>
-        </geometry>
-        <material name="LightGrey">
-          <color rgba="0.7 0.7 0.7 1.0"/>
-        </material>
-      </visual>
-      <collision>
-        <geometry>
-          <mesh filename="package://ur_description/meshes/ur10/collision/wrist2.stl"/>
-        </geometry>
-      </collision>
-      <xacro:cylinder_inertial radius="0.075" length="0.12" mass="${right_wrist_2_mass}">
+          <mesh filename="package://ur_description/meshes/ur5/visual/wrist2.dae" />
+        </geometry>
+        <material name="LightGrey">
+          <color rgba="0.7 0.7 0.7 1.0"/>
+        </material>
+      </visual>
+      <collision>
+        <geometry>
+          <mesh filename="package://ur_description/meshes/ur5/collision/wrist2.stl" />
+        </geometry>
+      </collision>
+      <xacro:cylinder_inertial radius="0.6" length="0.12" mass="${ur5_wrist_2_mass}">
         <origin xyz="0.0 0.0 0.0" rpy="0 0 0" />
       </xacro:cylinder_inertial>
@@ -231,11 +246,11 @@
       <parent link="${prefix}wrist_2_link" />
       <child link = "${prefix}wrist_3_link" />
-      <origin xyz="0.0 0.0 ${right_wrist_2_length}" rpy="0.0 0.0 0.0" />
+      <origin xyz="0.0 0.0 ${ur5_wrist_2_length}" rpy="0.0 0.0 0.0" />
       <axis xyz="0 1 0" />
       <xacro:unless value="${joint_limited}">
-        <limit lower="${-2.0 * pi}" upper="${2.0 * pi}" effort="54.0" velocity="3.2"/>
-      </xacro:unless>
-      <xacro:if value="${joint_limited}">
-        <limit lower="${-pi}" upper="${pi}" effort="54.0" velocity="3.2"/>
+        <limit lower="${-2.0 * pi}" upper="${2.0 * pi}" effort="28.0" velocity="3.2"/>
+      </xacro:unless>
+      <xacro:if value="${joint_limited}">
+        <limit lower="${-pi}" upper="${pi}" effort="28.0" velocity="3.2"/>
       </xacro:if>
       <dynamics damping="0.0" friction="0.0"/>
@@ -244,16 +259,16 @@
       <visual>
         <geometry>
-          <mesh filename="package://ur_description/meshes/ur10/visual/wrist3.dae"/>
-        </geometry>
-        <material name="LightGrey">
-          <color rgba="0.7 0.7 0.7 1.0"/>
-        </material>
-      </visual>
-      <collision>
-        <geometry>
-          <mesh filename="package://ur_description/meshes/ur10/collision/wrist3.stl"/>
-        </geometry>
-      </collision>
-      <xacro:cylinder_inertial radius="0.075" length="0.12" mass="${right_wrist_3_mass}">
+          <mesh filename="package://ur_description/meshes/ur5/visual/wrist3.dae" />
+        </geometry>
+        <material name="LightGrey">
+          <color rgba="0.7 0.7 0.7 1.0"/>
+        </material>
+      </visual>
+      <collision>
+        <geometry>
+          <mesh filename="package://ur_description/meshes/ur5/collision/wrist3.stl" />
+        </geometry>
+      </collision>
+      <xacro:cylinder_inertial radius="0.6" length="0.12" mass="${ur5_wrist_3_mass}">
         <origin xyz="0.0 0.0 0.0" rpy="0 0 0" />
       </xacro:cylinder_inertial>
@@ -262,5 +277,5 @@
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