Commit message: Change ur5 to left

File: dual_arm_robot_description/urdf/dual_arm_robot.urdf.xacro (robot description, xacro)
@@ -3,8 +3,7 @@
        name="dual_arm_robot">
   <xacro:property name="pi" value="3.1415926535897931"/>
-  <xacro:arg name="prefix_ur5" default="ur5_"/>
+  <xacro:arg name="prefix_left" default="left_"/>
   <xacro:arg name="prefix_right" default="right_"/>
-  <xacro:arg name="limited_ur5" default="true"/>
-  <xacro:arg name="limited_right" default="true"/>
+  <xacro:arg name="limited" default="true"/>
   <!-- common stuff -->
   <xacro:include filename="$(find ur_description)/urdf/common.gazebo.xacro"/>
@@ -27,26 +26,26 @@
   </joint>
   <!-- place ur5 arm -->
-  <xacro:ur5_robot prefix="$(arg prefix_ur5)" joint_limited="$(arg limited_ur5)"/>
-  <joint name="$(arg prefix_ur5)platform_mount" type="fixed">
-    <parent link="$(arg prefix_ur5)table_platform"/>
-    <child link ="$(arg prefix_ur5)base_link"/>
+  <xacro:ur5_robot prefix="$(arg prefix_left)" joint_limited="$(arg limited)"/>
+  <joint name="$(arg prefix_left)platform_mount" type="fixed">
+    <parent link="$(arg prefix_left)table_platform"/>
+    <child link ="$(arg prefix_left)base_link"/>
     <origin xyz="0.2745 -0.2405 0.2535" rpy="0 0 -${pi/2}" />
   </joint>
   <!-- place ur5 endeffector -->
-  <xacro:endeffector prefix="$(arg prefix_ur5)"/>
-  <joint name="$(arg prefix_ur5)ee_mount" type="fixed">
-    <parent link="$(arg prefix_ur5)ee_link" />
-    <child link = "$(arg prefix_ur5)ee_frame" />
+  <xacro:endeffector prefix="$(arg prefix_left)"/>
+  <joint name="$(arg prefix_left)ee_mount" type="fixed">
+    <parent link="$(arg prefix_left)ee_link" />
+    <child link = "$(arg prefix_left)ee_frame" />
     <origin xyz="0.0 0.0 0.0" rpy="${pi/2.0} 0.0 ${pi/2.0}" />
   </joint>
 <!--
-  <joint name="$(arg prefix_ur5)ee_mount" type="fixed">
-    <parent link="$(arg prefix_ur5)tool0"/>
-    <child link ="$(arg prefix_ur5)ee_frame"/>
+  <joint name="$(arg prefix_left)ee_mount" type="fixed">
+    <parent link="$(arg prefix_left)tool0"/>
+    <child link ="$(arg prefix_left)ee_frame"/>
     <origin xyz="0 0 0" rpy="0 0 ${pi}" />
   </joint>
 -->
   <!-- place ur10 arm -->
-  <xacro:right_robot prefix="$(arg prefix_right)" joint_limited="$(arg limited_right)"/>
+  <xacro:right_robot prefix="$(arg prefix_right)" joint_limited="$(arg limited)"/>
   <joint name="$(arg prefix_right)platform_mount" type="fixed">
     <parent link="$(arg prefix_right)table_platform"/>

File: dual_arm_robot_description/urdf/table.urdf.xacro (robot description, xacro)
@@ -121,5 +121,5 @@
     <origin xyz="0.84 0.019 0.04"/>
   </joint>
-  <link name="$(arg prefix_ur5)table_platform">
+  <link name="$(arg prefix_left)table_platform">
     <visual>
       <geometry>
@@ -137,7 +137,7 @@
     </collision>
   </link>
-  <joint name="$(arg prefix_ur5)table_ground_to_platform" type="fixed">
+  <joint name="$(arg prefix_left)table_ground_to_platform" type="fixed">
     <parent link="table_ground"/>
-    <child link="$(arg prefix_ur5)table_platform"/>
+    <child link="$(arg prefix_left)table_platform"/>
     <origin xyz="0 0 0"/>
   </joint>

Commit message: Change table_ground to stand_stand and edit the stand
Now the stand model in urdf is consistent with the real one

File: dual_arm_robot_description/urdf/dual_arm_robot.urdf.xacro (robot description, xacro)
@@ -10,25 +10,94 @@
   <!-- ur5 -->
   <xacro:include filename="$(find dual_arm_robot_description)/urdf/ur5.urdf.xacro"/> <!-- file has been edited because of same variable names in ur5 and ur10 -->
-  <!-- ur10 -->
-  <xacro:include filename="$(find dual_arm_robot_description)/urdf/ur5_right.urdf.xacro"/> <!-- original file has been edited because of same variable names in ur5 and ur10 -->
   <!-- endeffector -->
   <xacro:include filename="$(find dual_arm_robot_description)/urdf/endeffector.urdf.xacro"/>
-  <!-- table -->
+  <!-- table
   <xacro:include filename="$(find dual_arm_robot_description)/urdf/table.urdf.xacro"/>
+-->
   <!-- place table -->
   <xacro:table/>
-  <!-- place world reference -->
+  <xacro:property name="robot_horizontal_stand_width" value="0.5"/>
+	<xacro:property name="robot_vertical_stand_height" value="1.2"/>
+	<!-- color macros -->
+	<xacro:macro name="material_orange_transparent">
+		<material name="orange_transparent">
+			<color rgba="1 0.5 0 0.4"/>
+		</material>
+	</xacro:macro>
+	<xacro:macro name="material_blue_transparent">
+		<material name="blue_transparent">
+			<color rgba="0 0.8 1 0.4"/>
+		</material>
+	</xacro:macro>
+	<xacro:material_orange_transparent />
+	<xacro:material_blue_transparent />
+  <!-- end of color macros -->
+  <!-- Stand macros -->
+  <link name="stand1">
+		<visual>
+		<geometry>
+		<cylinder radius="0.0735" length="${robot_vertical_stand_height+0.2}"/>
+		</geometry>
+		<material name="orange_transparent"/>
+		</visual>
+		<collision>
+		<geometry>
+		<cylinder radius="0.0735" length="${robot_vertical_stand_height+0.2}"/>
+		</geometry>
+		<material name="blue_transparent"/>
+		</collision>
+	</link>
+	<link name="stand2">
+		<visual>
+		<geometry>
+		<cylinder radius="0.0735" length="${robot_horizontal_stand_width}"/>
+		</geometry>
+		<material name="orange_transparent"/>
+		</visual>
+		<collision>
+		<geometry>
+		<cylinder radius="0.0735" length="${robot_horizontal_stand_width}"/>
+		</geometry>
+		<material name="blue_transparent"/>
+		</collision>
+	</link>
+  <!-- End of stand macros-->
+  <!-- Place the stand in the world -->
   <link name="world"/>
-  <joint name="world_joint" type="fixed">
-    <parent link="world"/>
-    <child link ="table_ground"/>
-    <origin xyz="0.0 0.0 0.0" rpy="0.0 0.0 0.0" />
-  </joint>
-  <!-- place ur5 arm -->
+  <link name="stand_ground"/>
+    <!-- place world reference -->
+	<joint name="world_to_stand_ground" type="fixed">
+		<parent link="world"/>
+		<child link="stand_ground"/>
+		<origin xyz="0 0 0" rpy="0 0 0"/>
+	</joint>
+	<joint name="base_link_to_stand" type="fixed">
+		<parent link="stand_ground"/>
+		<child link="stand1"/>
+		<origin xyz="0 0 ${robot_vertical_stand_height/2}" rpy="0 0 0"/>
+	</joint>
+	<joint name="stand1_to_stand2" type="fixed">
+		<parent link="stand1"/>
+		<child link="stand2"/>
+		<origin xyz="0 0 ${robot_vertical_stand_height/2}" rpy="1.57 1.57 0"/>
+	</joint>
+<!--
+	<joint name="stand2_to_stand3" type="fixed">
+		<parent link="stand2"/>
+		<child link="stand3"/>
+		<origin xyz="-0.05 0 ${(robot_horizontal_stand_width/4)+0.15}" rpy="0 1.57 0"/>
+	</joint>
+	<joint name="stand2_to_stand4" type="fixed">
+		<parent link="stand2"/>
+		<child link="stand4"/>
+		<origin xyz="-0.05 0 -${(robot_horizontal_stand_width/4)+0.15}" rpy="0 1.57 0"/>
+	</joint>
+-->
+  <!-- place ur5 left arm    -->
   <xacro:ur5_robot prefix="$(arg prefix_left)" joint_limited="$(arg limited)"/>
-  <joint name="$(arg prefix_left)platform_mount" type="fixed">
-    <parent link="$(arg prefix_left)table_platform"/>
+  <joint name="stand2_to_left_arm" type="fixed">
+    <parent link="stand2"/>
     <child link ="$(arg prefix_left)base_link"/>
-    <origin xyz="0.2745 -0.2405 0.2535" rpy="0 0 -${pi/2}" />
+   <origin xyz="0 0 ${(robot_horizontal_stand_width/2)}" rpy="${pi/4.0} 0 0"/>
   </joint>
   <!-- place ur5 endeffector -->
@@ -46,12 +115,12 @@
   </joint>
 -->
-  <!-- place ur10 arm -->
-  <xacro:right_robot prefix="$(arg prefix_right)" joint_limited="$(arg limited)"/>
-  <joint name="$(arg prefix_right)platform_mount" type="fixed">
-    <parent link="$(arg prefix_right)table_platform"/>
+  <!-- place ur5 right arm  -->
+  <xacro:ur5_robot prefix="$(arg prefix_right)" joint_limited="$(arg limited)"/>
+  <joint name="stand2_to_right_arm" type="fixed">
+    <parent link="stand2"/>
     <child link ="$(arg prefix_right)base_link"/>
-    <origin xyz="0.1341 -0.3049 0.0155" rpy="0 0 ${pi/2}" />
+    <origin xyz="0 0 -${(robot_horizontal_stand_width/2)}" rpy="${pi/4.0} ${pi} 0"/>
   </joint>
-  <!-- place ur10 endeffector -->
+  <!-- place ur5 right endeffector -->
   <xacro:endeffector prefix="$(arg prefix_right)"/>
   <joint name="$(arg prefix_right)ee_mount" type="fixed">

Commit message: Change some parameters and set up the table
Change left_last_goal_pose_ to left_current_pose_;
Remove stand_groud;
Set up the table and box size;
Change the joint constraints range.

File: dual_arm_robot_description/urdf/dual_arm_robot.urdf.xacro (robot description, xacro)
@@ -12,10 +12,4 @@
   <!-- endeffector -->
   <xacro:include filename="$(find dual_arm_robot_description)/urdf/endeffector.urdf.xacro"/>
-  <!-- table
-  <xacro:include filename="$(find dual_arm_robot_description)/urdf/table.urdf.xacro"/>
--->
-  <!-- place table
-  <xacro:table/>
--->
   <xacro:property name="robot_horizontal_stand_width" value="0.5"/>
 	<xacro:property name="robot_vertical_stand_height" value="1.2"/>
@@ -63,18 +57,31 @@
 		</collision>
 	</link>
+	<link name="table">
+		<visual>
+			<geometry>
+				<box size="0.8 1 0.87" />
+			</geometry>
+			<material name="orange_transparent"/>
+		</visual>
+		<collision>
+			<geometry>
+		<box size="0.8 1 0.8" />
+		</geometry>
+		<material name="blue_transparent"/>
+		</collision>
+	</link>
+  <joint name="table_joint" type="fixed" >
+    <parent link="world" />
+    <child link="table" />
+    <origin xyz="-1.1 0 0.45" rpy="0 0 0" />
+</joint>
   <!-- End of stand macros-->
   <!-- Place the stand in the world -->
   <link name="world"/>
-  <link name="stand_ground"/>
     <!-- place world reference -->
-	<joint name="world_to_stand_ground" type="fixed">
+	<joint name="world_to_stand1" type="fixed">
 		<parent link="world"/>
-		<child link="stand_ground"/>
-		<origin xyz="0 0 0" rpy="0 0 0"/>
-	</joint>
-	<joint name="base_link_to_stand" type="fixed">
-		<parent link="stand_ground"/>
 		<child link="stand1"/>
-		<origin xyz="0 0 ${robot_vertical_stand_height/2}" rpy="0 0 0"/>
+		<origin xyz="0 0 0.6" rpy="0 0 0"/>
 	</joint>
 	<joint name="stand1_to_stand2" type="fixed">
@@ -83,16 +90,11 @@
 		<origin xyz="0 0 ${robot_vertical_stand_height/2}" rpy="1.57 1.57 0"/>
 	</joint>
-<!--
-	<joint name="stand2_to_stand3" type="fixed">
-		<parent link="stand2"/>
-		<child link="stand3"/>
-		<origin xyz="-0.05 0 ${(robot_horizontal_stand_width/4)+0.15}" rpy="0 1.57 0"/>
+<!-- place a table
+  	<joint name="world_to_table" type="fixed">
+		<parent link="world"/>
+		<child link="table"/>
+		<origin xyz="-1 0 0.5" rpy="0 0 0"/>
 	</joint>
-	<joint name="stand2_to_stand4" type="fixed">
-		<parent link="stand2"/>
-		<child link="stand4"/>
-		<origin xyz="-0.05 0 -${(robot_horizontal_stand_width/4)+0.15}" rpy="0 1.57 0"/>
-	</joint>
--->
+	-->
   <!-- place ur5 left arm    -->
   <xacro:ur5_robot prefix="$(arg prefix_left)" joint_limited="$(arg limited)"/>

File: dual_arm_robot_description/urdf/table.urdf.xacro (robot description, xacro)
@@ -1,164 +1,193 @@
 <?xml version="1.0"?>
-<robot xmlns:sensor="http://playerstage.sourceforge.net/gazebo/xmlschema/#sensor"
+<robot name="table"
+       xmlns:xi="http://www.w3.org/2001/XInclude"
+       xmlns:gazebo="http://playerstage.sourceforge.net/gazebo/xmlschema/#gz"
+       xmlns:model="http://playerstage.sourceforge.net/gazebo/xmlschema/#model"
+       xmlns:sensor="http://playerstage.sourceforge.net/gazebo/xmlschema/#sensor"
+       xmlns:body="http://playerstage.sourceforge.net/gazebo/xmlschema/#body"
+       xmlns:geom="http://playerstage.sourceforge.net/gazebo/xmlschema/#geom"
+       xmlns:joint="http://playerstage.sourceforge.net/gazebo/xmlschema/#joint"
+       xmlns:interface="http://playerstage.sourceforge.net/gazebo/xmlschema/#interface"
+       xmlns:rendering="http://playerstage.sourceforge.net/gazebo/xmlschema/#rendering"
+       xmlns:renderable="http://playerstage.sourceforge.net/gazebo/xmlschema/#renderable"
        xmlns:controller="http://playerstage.sourceforge.net/gazebo/xmlschema/#controller"
-       xmlns:interface="http://playerstage.sourceforge.net/gazebo/xmlschema/#interface"
-       xmlns:xacro="http://ros.org/wiki/xacro">
+       xmlns:physics="http://playerstage.sourceforge.net/gazebo/xmlschema/#physics">
+  <property name="table_height" value="0.8" />
+  <property name="table_width" value="1.0" />
+  <property name="table_depth" value="1.0" />
+  <property name="leg_radius" value="0.02" />
+  <property name="table_x" value="0.98" />
+  <property name="table_y" value="0.0" />
+  <property name="table_z" value="0.0" />
+  <property name="table_top_thickness" value="0.05"/>
+  <property name="M_PI" value="3.1415926535897931" />
   <xacro:macro name="table">
-  <link name="table_ground">
+  <!-- tabletop height is .55+.01+.025=.585 -->
+  <link name="table_top_link">
+    <inertial>
+      <mass value="1.0" />
+      <origin xyz="${table_x} ${table_y} ${table_z+table_height-table_top_thickness/2}" />
+      <inertia ixx="1" ixy="0"  ixz="0"
+               iyy="1" iyz="0"
+               izz="1" />
+    </inertial>
     <visual>
+      <origin xyz="${table_x} ${table_y} ${table_z+table_height-table_top_thickness/2}" />
       <geometry>
-        <mesh filename="package://dual_arm_robot_description/meshes/table/table_ground.stl"/>
+        <box size="${table_width} ${table_depth} ${table_top_thickness}" />
       </geometry>
-      <material name="white">
-        <color rgba="1 1 1 1"/>
-      </material>
     </visual>
-    <origin rpy="0 0 0" xyz="0 0 0"/>
     <collision>
+      <origin xyz="${table_x} ${table_y} ${table_z+table_height-table_top_thickness/2}" />
       <geometry>
-        <mesh filename="package://dual_arm_robot_description/meshes/table/table_ground.stl"/>
+        <box size="${table_width} ${table_depth} ${table_top_thickness}" />
       </geometry>
     </collision>
   </link>
-  <link name="table_side_left">
+  <gazebo reference="table_top_link">
+    <material>Gazebo/LightWood</material>
+    <mu1>50.0</mu1>
+    <mu2>50.0</mu2>
+    <kp>1000000.0</kp>
+    <kd>1.0</kd>
+  </gazebo>
+  <joint name="leg1_joint" type="fixed" >
+    <parent link="table_top_link" />
+    <origin xyz="${table_x+table_width/2} ${table_y+table_depth/2} ${table_z+table_height}" rpy="0 0 0" />
+    <child link="leg1_link" />
+  </joint>
+  <link name="leg1_link">
+    <inertial>
+      <mass value="1.0" />
+      <origin xyz="0 0 ${-table_height/2}" />
+      <inertia ixx="0.1" ixy="0"  ixz="0"
+               iyy="0.1" iyz="0"
+               izz="0.01" />
+    </inertial>
     <visual>
+      <origin xyz="0.0 0.0 ${-table_height/2}" rpy="0 0 0" />
       <geometry>
-        <mesh filename="package://dual_arm_robot_description/meshes/table/table_side.stl"/>
+        <cylinder radius="${leg_radius}" length="${table_height}" />
       </geometry>
-      <material name="glass">
-        <color rgba="0 0 1 0.5"/>
-      </material>
     </visual>
-    <origin rpy="0 0 0" xyz="0 0 0"/>
     <collision>
+      <origin xyz="0.0 0.0 ${-table_height/2}" rpy="0.0 0.0 0.0" />
       <geometry>
-        <mesh filename="package://dual_arm_robot_description/meshes/table/table_side.stl"/>
+        <cylinder radius="${leg_radius}" length="${table_height}" />
       </geometry>
     </collision>
   </link>
-  <joint name="table_ground_to_side_left" type="fixed">
-    <parent link="table_ground"/>
-    <child link="table_side_left"/>
-    <origin xyz="0 0 0"/>
+  <gazebo reference="leg1_link">
+    <material>Gazebo/Red</material>
+    <mu1>1000.0</mu1>
+    <mu2>1000.0</mu2>
+    <kp>10000000.0</kp>
+    <kd>1.0</kd>
+    <selfCollide>true</selfCollide>
+  </gazebo>
+  <joint name="leg2_joint" type="fixed" >
+    <parent link="table_top_link" />
+    <origin xyz="${table_x-table_width/2} ${table_y+table_depth/2} ${table_z+table_height}" rpy="0 0 0" />
+    <child link="leg2_link" />
   </joint>
-  <link name="table_side_right">
+  <link name="leg2_link">
+    <inertial>
+      <mass value="1.0" />
+      <origin xyz="0 0 ${-table_height/2}" />
+      <inertia ixx="0.1" ixy="0"  ixz="0"
+               iyy="0.1" iyz="0"
+               izz="0.01" />
+    </inertial>
     <visual>
+      <origin xyz="0.0 0.0 ${-table_height/2}" rpy="0 0 0" />
       <geometry>
-        <mesh filename="package://dual_arm_robot_description/meshes/table/table_side.stl"/>
+        <cylinder radius="${leg_radius}" length="${table_height}" />
       </geometry>
-      <material name="glass"/>
     </visual>
-    <origin rpy="0 0 0" xyz="0 0 0"/>
     <collision>
+      <origin xyz="0.0 0.0 ${-table_height/2}" rpy="0.0 0.0 0.0" />
       <geometry>
-        <mesh filename="package://dual_arm_robot_description/meshes/table/table_side.stl"/>
+        <cylinder radius="${leg_radius}" length="${table_height}" />
       </geometry>
     </collision>
   </link>
-  <joint name="table_ground_to_side_right" type="fixed">
-    <parent link="table_ground"/>
-    <child link="table_side_right"/>
-    <origin xyz="1.585 0 0"/>
+  <gazebo reference="leg2_link">
+    <material>Gazebo/Red</material>
+    <mu1>1000.0</mu1>
+    <mu2>1000.0</mu2>
+    <kp>10000000.0</kp>
+    <kd>1.0</kd>
+    <selfCollide>true</selfCollide>
+  </gazebo>
+  <joint name="leg3_joint" type="fixed" >
+    <parent link="table_top_link" />
+    <origin xyz="${table_x+table_width/2} ${table_y-table_depth/2} ${table_z+table_height}" rpy="0 0 0" />
+    <child link="leg3_link" />
   </joint>
-  <link name="table_back">
+  <link name="leg3_link">
+    <inertial>
+      <mass value="1.0" />
+      <origin xyz="0 0 ${-table_height/2}" />
+      <inertia ixx="0.1" ixy="0"  ixz="0"
+               iyy="0.1" iyz="0"
+               izz="0.01" />
+    </inertial>
     <visual>
+      <origin xyz="0.0 0.0 ${-table_height/2}" rpy="0 0 0" />
       <geometry>
-        <mesh filename="package://dual_arm_robot_description/meshes/table/table_back.stl"/>
+        <cylinder radius="${leg_radius}" length="${table_height}" />
       </geometry>
-    <material name="white"/>
     </visual>
-    <origin rpy="0 0 0" xyz="0 0 0"/>
     <collision>
+      <origin xyz="0.0 0.0 ${-table_height/2}" rpy="0.0 0.0 0.0" />
       <geometry>
-        <mesh filename="package://dual_arm_robot_description/meshes/table/table_back.stl"/>
+        <cylinder radius="${leg_radius}" length="${table_height}" />
       </geometry>
     </collision>
   </link>
-  <joint name="table_ground_to_back" type="fixed">
-    <parent link="table_ground"/>
-    <child link="table_back"/>
-    <origin xyz="0 0 0"/>
+  <gazebo reference="leg3_link">
+    <material>Gazebo/Red</material>
+    <mu1>1000.0</mu1>
+    <mu2>1000.0</mu2>
+    <kp>10000000.0</kp>
+    <kd>1.0</kd>
+    <selfCollide>true</selfCollide>
+  </gazebo>
+  <joint name="leg4_joint" type="fixed" >
+    <parent link="table_top_link" />
+    <origin xyz="${table_x-table_width/2} ${table_y-table_depth/2} ${table_z+table_height}" rpy="0 0 0" />
+    <child link="leg4_link" />
   </joint>
-  <link name="table_front">
+  <link name="leg4_link">
+    <inertial>
+      <mass value="1.0" />
+      <origin xyz="0 0 ${-table_height/2}" />
+      <inertia ixx="0.1" ixy="0"  ixz="0"
+               iyy="0.1" iyz="0"
+               izz="0.01" />
+    </inertial>
     <visual>
+      <origin xyz="0.0 0.0 ${-table_height/2}" rpy="0 0 0" />
       <geometry>
-        <mesh filename="package://dual_arm_robot_description/meshes/table/table_front.stl"/>
+        <cylinder radius="${leg_radius}" length="${table_height}" />
       </geometry>
-    <material name="glass"/>
     </visual>
-    <origin rpy="0 0 0" xyz="0 0 0"/>
     <collision>
+      <origin xyz="0.0 0.0 ${-table_height/2}" rpy="0.0 0.0 0.0" />
       <geometry>
-        <mesh filename="package://dual_arm_robot_description/meshes/table/table_front.stl"/>
+        <cylinder radius="${leg_radius}" length="${table_height}" />
       </geometry>
     </collision>
   </link>
-  <joint name="table_ground_to_front" type="fixed">
-    <parent link="table_ground"/>
-    <child link="table_front"/>
-    <origin xyz="0 -1.319 0"/>
-  </joint>
-  <link name="table_camerahanger">
-    <visual>
-      <geometry>
-        <mesh filename="package://dual_arm_robot_description/meshes/table/table_camerahanger.stl"/>
-      </geometry>
-    <material name="aluminium">
-      <color rgba="0.5 0.5 0.5 1"/>
-    </material>
-    </visual>
-    <origin rpy="0 0 0" xyz="0 0 0"/>
-    <collision>
-      <geometry>
-        <mesh filename="package://dual_arm_robot_description/meshes/table/table_camerahanger.stl"/>
-      </geometry>
-    </collision>
-  </link>
-  <joint name="table_ground_to_camerahanger" type="fixed">
-    <parent link="table_ground"/>
-    <child link="table_camerahanger"/>
-<!--origin xyz="0.8 0.019 0"-->
-    <origin xyz="0.84 0.019 0.04"/>
-  </joint>
-  <link name="$(arg prefix_left)table_platform">
-    <visual>
-      <geometry>
-        <mesh filename="package://dual_arm_robot_description/meshes/table/table_platform_ur5.stl"/>
-      </geometry>
-    <material name="steel">
-      <color rgba="0.4 0.4 0.4 1"/>
-    </material>
-    </visual>
-    <origin rpy="0 0 0" xyz="0 0 0"/>
-    <collision>
-      <geometry>
-        <mesh filename="package://dual_arm_robot_description/meshes/table/table_platform_ur5.stl"/>
-      </geometry>
-    </collision>
-  </link>
-  <joint name="$(arg prefix_left)table_ground_to_platform" type="fixed">
-    <parent link="table_ground"/>
-    <child link="$(arg prefix_left)table_platform"/>
-    <origin xyz="0 0 0"/>
-  </joint>
-  <link name="$(arg prefix_right)table_platform">
-    <visual>
-      <geometry>
-        <mesh filename="package://dual_arm_robot_description/meshes/table/table_platform_right.stl"/>
-      </geometry>
-    <material name="steel"/>
-    </visual>
-    <origin rpy="0 0 0" xyz="0 0 0"/>
-    <collision>
-      <geometry>
-        <mesh filename="package://dual_arm_robot_description/meshes/table/table_platform_right.stl"/>
-      </geometry>
-    </collision>
-  </link>
-  <joint name="$(arg prefix_right)table_ground_to_platform" type="fixed">
-    <parent link="table_ground"/>
-    <child link="$(arg prefix_right)table_platform"/>
-    <origin xyz="1.076 0 0"/>
-  </joint>
-  </xacro:macro>
+  <gazebo reference="leg4_link">
+    <material>Gazebo/Red</material>
+    <mu1>1000.0</mu1>
+    <mu2>1000.0</mu2>
+    <kp>10000000.0</kp>
+    <kd>1.0</kd>
+    <selfCollide>true</selfCollide>
+  </gazebo>
+  <gazebo>
+    <canonicalBody>table_top_link</canonicalBody>
+  </gazebo>
 </robot>
