Commit message: Create getPositionIK()
Create a function to compute IK. It should be noted that  robot_state::RobotState contains two arms. Should think about how to deal with it.

File: dual_arm_robot_description/urdf/dual_arm_robot.urdf.xacro (robot description, xacro)
@@ -60,5 +60,5 @@
 		<visual>
 			<geometry>
-				<box size="0.8 1 0.87" />
+				<box size="0.8 1 0.94" />
 			</geometry>
 			<material name="orange_transparent"/>
@@ -66,5 +66,5 @@
 		<collision>
 			<geometry>
-		<box size="0.8 1 0.8" />
+		<box size="1 1 1" />
 		</geometry>
 		<material name="blue_transparent"/>
@@ -74,5 +74,5 @@
     <parent link="world" />
     <child link="table" />
-    <origin xyz="-1.1 0 0.45" rpy="0 0 0" />
+    <origin xyz="-1.1 0 0.47" rpy="0 0 0" />
 </joint>
   <!-- End of stand macros-->

File: dual_arm_robot_description/urdf/ur5.urdf.xacro (robot description, xacro)
@@ -296,5 +296,5 @@
                  degrees)
       -->
-      <origin xyz="0 0 0" rpy="0 0 ${-pi}"/>
+      <origin xyz="0 0 0" rpy="0 0 ${pi}"/>
       <parent link="${prefix}base_link"/>
       <child link="${prefix}base"/>
@@ -303,5 +303,5 @@
     <link name="${prefix}tool0"/>
     <joint name="${prefix}wrist_3_link-tool0_fixed_joint" type="fixed">
-      <origin xyz="0 ${ur5_wrist_3_length} 0" rpy="${pi/-2.0} 0 0"/>
+      <origin xyz="0 ${ur5_wrist_3_length} 0" rpy="${pi/-2.0} ${2*pi} 0"/>
       <parent link="${prefix}wrist_3_link"/>
       <child link="${prefix}tool0"/>

Commit message: Put the kinematic set-up stuffs into class
robotModelLoader, kinematic_model, kinematic_state, left_joint_model_group

File: dual_arm_robot_description/urdf/dual_arm_robot.urdf.xacro (robot description, xacro)
@@ -66,5 +66,5 @@
 		<collision>
 			<geometry>
-		<box size="1 1 1" />
+			<box size="1 1 0.95" />
 		</geometry>
 		<material name="blue_transparent"/>

Commit message: Added some helper functions and adjusted the urdf files.
The pose in ROS now is consistent with the  one in smartPad.
It should be noted that the base and tip link are left_base and left_ee_link ,respectively. The same thing to the right arm.
In smartPad, the Feature should be choosen BASE, and Rotation is RPY[rad].

File: dual_arm_robot_description/urdf/dual_arm_robot.urdf.xacro (robot description, xacro)
@@ -1,5 +1,6 @@
-<?xml version="1.0"?>
+<?xml version="1.0"?> <!--this tag must be in the first line of the xml files-->
 <robot xmlns:xacro="http://www.ros.org/wiki/xacro"
        name="dual_arm_robot">
+<!-- rosrun xacro xacro.py dual_arm_robot.urdf.xacro >  dual_arm_robot.urdf -->
   <xacro:property name="pi" value="3.1415926535897931"/>
   <xacro:arg name="prefix_left" default="left_"/>
@@ -10,6 +11,7 @@
   <!-- ur5 -->
   <xacro:include filename="$(find dual_arm_robot_description)/urdf/ur5.urdf.xacro"/> <!-- file has been edited because of same variable names in ur5 and ur10 -->
-  <!-- endeffector -->
+  <!-- endeffector
   <xacro:include filename="$(find dual_arm_robot_description)/urdf/endeffector.urdf.xacro"/>
+-->
   <xacro:property name="robot_horizontal_stand_width" value="0.5"/>
 	<xacro:property name="robot_vertical_stand_height" value="1.2"/>
@@ -32,5 +34,5 @@
 		<visual>
 		<geometry>
-		<cylinder radius="0.0735" length="${robot_vertical_stand_height+0.2}"/>
+		<cylinder radius="0.0735" length="0.5"/>
 		</geometry>
 		<material name="orange_transparent"/>
@@ -38,5 +40,5 @@
 		<collision>
 		<geometry>
-		<cylinder radius="0.0735" length="${robot_vertical_stand_height+0.2}"/>
+		<cylinder radius="0.0735" length="0.5"/>
 		</geometry>
 		<material name="blue_transparent"/>
@@ -57,8 +59,22 @@
 		</collision>
 	</link>
+<link name="stand_Base">
+		<visual>
+		<geometry>
+		<cylinder radius="0.5" length="0.7"/>
+		</geometry>
+		<material name="orange_transparent"/>
+		</visual>
+		<collision>
+		<geometry>
+		<cylinder radius="0.5" length="0.7"/>
+		</geometry>
+		<material name="blue_transparent"/>
+		</collision>
+	</link>
 	<link name="table">
 		<visual>
 			<geometry>
-				<box size="0.8 1 0.94" />
+				<box size="1 1.2 0.92" />
 			</geometry>
 			<material name="orange_transparent"/>
@@ -66,5 +82,5 @@
 		<collision>
 			<geometry>
-			<box size="1 1 0.95" />
+		<box size="1 1.2 0.92" />
 		</geometry>
 		<material name="blue_transparent"/>
@@ -74,5 +90,5 @@
     <parent link="world" />
     <child link="table" />
-    <origin xyz="-1.1 0 0.47" rpy="0 0 0" />
+    <origin xyz="-1 0 0.46" rpy="0 0 0" />
 </joint>
   <!-- End of stand macros-->
@@ -80,6 +96,11 @@
   <link name="world"/>
     <!-- place world reference -->
-	<joint name="world_to_stand1" type="fixed">
+  <joint name="world_to_stand_Base" type="fixed">
 		<parent link="world"/>
+		<child link="stand_Base"/>
+		<origin xyz="0 0 0.35" rpy="0 0 0"/>
+	</joint>
+	<joint name="Base_to_stand1" type="fixed">
+		<parent link="stand_Base"/>
 		<child link="stand1"/>
 		<origin xyz="0 0 0.6" rpy="0 0 0"/>
@@ -88,5 +109,5 @@
 		<parent link="stand1"/>
 		<child link="stand2"/>
-		<origin xyz="0 0 ${robot_vertical_stand_height/2}" rpy="1.57 1.57 0"/>
+		<origin xyz="0 0 0.25" rpy="1.57 1.57 0"/>
 	</joint>
 <!-- place a table

File: dual_arm_robot_description/urdf/ur5.urdf.xacro (robot description, xacro)
@@ -97,5 +97,5 @@
       </xacro:unless>
       <xacro:if value="${joint_limited}">
-        <limit lower="${-2*pi}" upper="${2*pi}" effort="150.0" velocity="3.15"/>
+        <limit lower="${-pi}" upper="${pi}" effort="150.0" velocity="3.15"/>
       </xacro:if>
       <dynamics damping="0.0" friction="0.0"/>
@@ -159,5 +159,5 @@
       </xacro:unless>
       <xacro:if value="${joint_limited}">
-        <limit lower="${-2*pi}" upper="${2*pi}" effort="150.0" velocity="3.15"/>
+        <limit lower="${-pi}" upper="${pi}" effort="150.0" velocity="3.15"/>
       </xacro:if>
       <dynamics damping="0.0" friction="0.0"/>
@@ -190,5 +190,5 @@
       </xacro:unless>
       <xacro:if value="${joint_limited}">
-        <limit lower="${-2*pi}" upper="${2*pi}" effort="28.0" velocity="3.2"/>
+        <limit lower="${-pi}" upper="${pi}" effort="28.0" velocity="3.2"/>
       </xacro:if>
       <dynamics damping="0.0" friction="0.0"/>
@@ -221,5 +221,5 @@
       </xacro:unless>
       <xacro:if value="${joint_limited}">
-        <limit lower="${-2*pi}" upper="${2*pi}" effort="28.0" velocity="3.2"/>
+        <limit lower="${-pi}" upper="${pi}" effort="28.0" velocity="3.2"/>
       </xacro:if>
       <dynamics damping="0.0" friction="0.0"/>
@@ -249,8 +249,8 @@
       <axis xyz="0 1 0" />
       <xacro:unless value="${joint_limited}">
-        <limit lower="${-2.0 * pi}" upper="${2.0 * pi}" effort="28.0" velocity="3.2"/>
-      </xacro:unless>
-      <xacro:if value="${joint_limited}">
-        <limit lower="${-2*pi}" upper="${2*pi}" effort="28.0" velocity="3.2"/>
+        <limit lower="${-pi}" upper="${pi}" effort="28.0" velocity="3.2"/>
+      </xacro:unless>
+      <xacro:if value="${joint_limited}">
+        <limit lower="${-pi}" upper="${pi}" effort="28.0" velocity="3.2"/>
       </xacro:if>
       <dynamics damping="0.0" friction="0.0"/>
@@ -277,5 +277,5 @@
       <parent link="${prefix}wrist_3_link" />
       <child link = "${prefix}ee_link" />
-      <origin xyz="0.0 ${ur5_wrist_3_length} 0.0" rpy="0.0 0.0 ${pi/2.0}" />
+      <origin xyz="0.0 ${ur5_wrist_3_length} 0.0" rpy="${pi/2} ${pi} ${-pi}" />
     </joint>
     <link name="${prefix}ee_link">
@@ -296,15 +296,17 @@
                  degrees)
       -->
-      <origin xyz="0 0 0" rpy="0 0 ${pi}"/>
+      <origin xyz="0 0 0" rpy="0 0 ${-pi}"/>
       <parent link="${prefix}base_link"/>
       <child link="${prefix}base"/>
     </joint>
     <!-- Frame coincident with all-zeros TCP on UR controller -->
+    <!--
     <link name="${prefix}tool0"/>
     <joint name="${prefix}wrist_3_link-tool0_fixed_joint" type="fixed">
-      <origin xyz="0 ${ur5_wrist_3_length} 0" rpy="${pi/-2.0} ${2*pi} 0"/>
+      <origin xyz="0 ${ur5_wrist_3_length} 0" rpy="${pi/-2.0} 0 0"/>
       <parent link="${prefix}wrist_3_link"/>
       <child link="${prefix}tool0"/>
     </joint>
+    -->
   </xacro:macro>
 </robot>

Commit message: Log Cartesian data

File: dual_arm_robot_description/urdf/dual_arm_robot.urdf.xacro (robot description, xacro)
@@ -10,5 +10,5 @@
   <xacro:include filename="$(find ur_description)/urdf/common.gazebo.xacro"/>
   <!-- ur5 -->
-  <xacro:include filename="$(find dual_arm_robot_description)/urdf/ur5.urdf.xacro"/> <!-- file has been edited because of same variable names in ur5 and ur10 -->
+  <xacro:include filename="$(find dual_arm_robot_description)/urdf/ur5.urdf.xacro"/>
   <!-- endeffector
   <xacro:include filename="$(find dual_arm_robot_description)/urdf/endeffector.urdf.xacro"/>
@@ -34,5 +34,5 @@
 		<visual>
 		<geometry>
-		<cylinder radius="0.0735" length="0.5"/>
+		<cylinder radius="0.08" length="0.8"/>
 		</geometry>
 		<material name="orange_transparent"/>
@@ -40,5 +40,5 @@
 		<collision>
 		<geometry>
-		<cylinder radius="0.0735" length="0.5"/>
+		<cylinder radius="0.08" length="0.8"/>
 		</geometry>
 		<material name="blue_transparent"/>
@@ -48,5 +48,5 @@
 		<visual>
 		<geometry>
-		<cylinder radius="0.0735" length="${robot_horizontal_stand_width}"/>
+		<cylinder radius="0.08" length="${robot_horizontal_stand_width}"/>
 		</geometry>
 		<material name="orange_transparent"/>
@@ -54,5 +54,5 @@
 		<collision>
 		<geometry>
-		<cylinder radius="0.0735" length="${robot_horizontal_stand_width}"/>
+		<cylinder radius="0.08" length="${robot_horizontal_stand_width}"/>
 		</geometry>
 		<material name="blue_transparent"/>

File: dual_arm_robot_description/urdf/ur5.urdf.xacro (robot description, xacro)
@@ -221,5 +221,5 @@
       </xacro:unless>
       <xacro:if value="${joint_limited}">
-        <limit lower="${-2*pi}" upper="${2*pi}" effort="28.0" velocity="2"/>
+        <limit lower="${-pi}" upper="${pi}" effort="28.0" velocity="2"/>
       </xacro:if>
       <dynamics damping="0.0" friction="0.0"/>
