Commit message: Realized the cartesian admittance controller

File: dual_arm_manipulation/dual_arm_robot_description/urdf/ur5.urdf.xacro (robot description, xacro)
@@ -306,5 +306,5 @@
     <link name="${prefix}tool0"/>
     <joint name="${prefix}wrist_3_link-tool0_fixed_joint" type="fixed">
-      <origin xyz="0 ${ur5_wrist_3_length} 0" rpy="${pi/-2.0} 0 0"/>
+      <origin xyz="0 ${ur5_wrist_3_length} 0" rpy="${pi/2.0} 0 0"/>
       <parent link="${prefix}wrist_3_link"/>
       <child link="${prefix}tool0"/>

Commit message: Edit the namespace for cartesian admittance controller

File: dual_arm_manipulation/dual_arm_robot_description/urdf/ur5.urdf.xacro (robot description, xacro)
@@ -306,5 +306,5 @@
     <link name="${prefix}tool0"/>
     <joint name="${prefix}wrist_3_link-tool0_fixed_joint" type="fixed">
-      <origin xyz="0 ${ur5_wrist_3_length} 0" rpy="${pi/2.0} 0 0"/>
+      <origin xyz="0 ${ur5_wrist_3_length} 0" rpy="${pi/-2.0} 0 0"/>
       <parent link="${prefix}wrist_3_link"/>
       <child link="${prefix}tool0"/>

Commit message: BE CAREFUL: The end effector frame has been changed.

File: dual_arm_manipulation/dual_arm_robot_description/urdf/ur5.urdf.xacro (robot description, xacro)
@@ -90,8 +90,12 @@
       </xacro:cylinder_inertial>
     </link>
+    <!--This connection is different from the original one (ur_description).
+        The parent link is changed from ${prefix}base_link to ${prefix}base,
+        then the transform from the base to tool0 is coincident with teachPad.
+        The joint rpy is adjusted to rpy="0 0 ${pi}", if connected to ${prefix}base_link, it should be rpy="0 0 0" -->
     <joint name="${prefix}shoulder_pan_joint" type="revolute">
-      <parent link="${prefix}base_link" />
+      <parent link="${prefix}base" />
       <child link = "${prefix}shoulder_link" />
-      <origin xyz="0.0 0.0 ${ur5_shoulder_height}" rpy="0.0 0.0 0.0" />
+      <origin xyz="0.0 0.0 ${ur5_shoulder_height}" rpy="0 0 ${pi}" />
       <axis xyz="0 0 1" />
       <xacro:unless value="${joint_limited}">
