Commit message: Reorganize folders and add ft300  and end-effectors in urdf
1. Reorganize the folders. Put all driver stuff in the project folder, then the customized changes could be kept. 
2. Add FT300 at the end of left arm.
3. Add end-effectors at the end of two arms.

File: dual_arm_manipulation/dual_arm_robot_description/urdf/dual_arm_robot.urdf.xacro (robot description, xacro)
@@ -11,7 +11,8 @@
   <!-- ur5 -->
   <xacro:include filename="$(find dual_arm_robot_description)/urdf/ur5.urdf.xacro"/>
-  <!-- endeffector
+  <!-- ft300 -->
+	<xacro:include filename="$(find robotiq_ft_sensor)/urdf/robotiq_fts300.urdf.xacro" />
+  <!-- endeffector -->
   <xacro:include filename="$(find dual_arm_robot_description)/urdf/endeffector.urdf.xacro"/>
--->
   <xacro:property name="robot_horizontal_stand_width" value="0.5"/>
 	<xacro:property name="robot_vertical_stand_height" value="1.2"/>
@@ -125,13 +126,19 @@
    <origin xyz="0 0 ${(robot_horizontal_stand_width/2)}" rpy="${pi/4.0} 0 0"/>
   </joint>
+  <!-- place robotiq_fts300 to left arm -->
+  <xacro:robotiq_fts300 prefix=""/>
+  <!-- mount the fts to the robot -->
+  <joint name="$(arg prefix_left)fts_fix" type="fixed" >
+    <origin xyz="0 0 0" rpy="0 1.57 0"/>
+    <parent link="$(arg prefix_left)ee_link" />
+    <child link="fts_robotside" />
+  </joint>
   <!-- place ur5 endeffector -->
-	<!--
   <xacro:endeffector prefix="$(arg prefix_left)"/>
   <joint name="$(arg prefix_left)ee_mount" type="fixed">
-    <parent link="$(arg prefix_left)ee_link" />
+    <parent link="fts_toolside" />
     <child link = "$(arg prefix_left)ee_frame" />
-    <origin xyz="0.0 0.0 0.0" rpy="${pi/2.0} 0.0 ${pi/2.0}" />
+    <origin xyz="0.0 0.0 0.0" rpy="0 0.0 0" />
   </joint>
-	-->
 <!--
   <joint name="$(arg prefix_left)ee_mount" type="fixed">
@@ -149,5 +156,4 @@
   </joint>
   <!-- place ur5 right endeffector -->
-	<!--
   <xacro:endeffector prefix="$(arg prefix_right)"/>
   <joint name="$(arg prefix_right)ee_mount" type="fixed">
@@ -156,5 +162,4 @@
     <origin xyz="0.0 0.0 0.0" rpy="${pi/2.0} 0.0 ${pi/2.0}" />
   </joint>
-	-->
 <!--
   <joint name="$(arg prefix_right)ee_mount" type="fixed">

Commit message: Add some  virtual walls
1. Add two virtual walls to limit the workspace.
2. Regenerate moveit configuration.

File: dual_arm_manipulation/dual_arm_robot_description/urdf/dual_arm_robot.urdf.xacro (robot description, xacro)
@@ -162,4 +162,61 @@
     <origin xyz="0.0 0.0 0.0" rpy="${pi/2.0} 0.0 ${pi/2.0}" />
   </joint>
+  	<link name="wall">
+		<visual>
+			<geometry>
+				<box size="1 1 3" />
+			</geometry>
+			<material name="blue_transparent"/>
+		</visual>
+		<collision>
+			<geometry>
+		<box size="1 1 3" />
+		</geometry>
+		<material name="blue_transparent"/>
+		</collision>
+	</link>
+  <joint name="wall_joint" type="fixed" >
+    <parent link="world" />
+    <child link="wall" />
+    <origin xyz="-1.6 -1.55 1.5" rpy="0 0 0" />
+</joint>
+<link name="wall1">
+		<visual>
+			<geometry>
+				<box size="0.01 2 3" />
+			</geometry>
+			<material name="blue_transparent"/>
+		</visual>
+		<collision>
+			<geometry>
+		<box size="0.01 2 3" />
+		</geometry>
+		<material name="blue_transparent"/>
+		</collision>
+	</link>
+  <joint name="wall_joint1" type="fixed" >
+    <parent link="world" />
+    <child link="wall1" />
+    <origin xyz="0.5 0 1.5" rpy="0 0 0" />
+</joint>
+<link name="wall2">
+		<visual>
+			<geometry>
+				<box size="2 0.01 3" />
+			</geometry>
+			<material name="blue_transparent"/>
+		</visual>
+		<collision>
+			<geometry>
+		<box size="2 0.01 3" />
+		</geometry>
+		<material name="blue_transparent"/>
+		</collision>
+	</link>
+  <joint name="wall_joint2" type="fixed" >
+    <parent link="world" />
+    <child link="wall2" />
+    <origin xyz="-1 1.4 1.5" rpy="0 0 0" />
+</joint>
 <!--
   <joint name="$(arg prefix_right)ee_mount" type="fixed">

Commit message: Adjust the urdf file
1. Increase the table height;
2. Change the grasp position;
3. Limit the joint_wrist3 in the range of pi;

File: dual_arm_manipulation/dual_arm_robot_description/urdf/dual_arm_robot.urdf.xacro (robot description, xacro)
@@ -77,5 +77,5 @@
 		<visual>
 			<geometry>
-				<box size="1 1.2 0.92" />
+				<box size="1 1.2 0.97" />
 			</geometry>
 			<material name="orange_transparent"/>
@@ -91,5 +91,5 @@
     <parent link="world" />
     <child link="table" />
-    <origin xyz="-1 0 0.46" rpy="0 0 0" />
+    <origin xyz="-1 0 0.485" rpy="0 0 0" />
 </joint>
   <!-- End of stand macros-->

File: dual_arm_manipulation/dual_arm_robot_description/urdf/ur5.urdf.xacro (robot description, xacro)
@@ -252,5 +252,5 @@
       </xacro:unless>
       <xacro:if value="${joint_limited}">
-        <limit lower="${-2*pi}" upper="${2*pi}" effort="28.0" velocity="2"/>
+        <limit lower="${-pi}" upper="${pi}" effort="28.0" velocity="2"/>
       </xacro:if>
       <dynamics damping="0.0" friction="0.0"/>

Commit message: Adjust the FT sensor and end-effector angles

File: dual_arm_manipulation/dual_arm_robot_description/urdf/dual_arm_robot.urdf.xacro (robot description, xacro)
@@ -135,10 +135,10 @@
   </joint>
 	-->
-  <!-- place ur5 endeffector -->
+  <!-- place ur5 endeffector  -->
   <xacro:endeffector prefix="$(arg prefix_left)"/>
   <joint name="$(arg prefix_left)ee_mount" type="fixed">
     <parent link="fts_toolside" />
     <child link = "$(arg prefix_left)ee_frame" />
-    <origin xyz="0.0 0.0 0.0" rpy="0 0.0 0" />
+    <origin xyz="0.0 0.0 0.0" rpy="0 0 0 " />
   </joint>
 <!--

File: robotiq/robotiq_force_torque_sensor/urdf/robotiq_fts300.urdf.xacro (robot description, xacro)
@@ -4,5 +4,5 @@
         <!-- mount the fts to the robot -->
         <joint name="${prefix}fts_fix" type="fixed" >
-            <origin xyz="0 0 -0.009" rpy="0 0 0"/>
+            <origin xyz="0 0 -0.009" rpy="0 1.57 0"/>
             <parent link="${parent}" />
             <child link="${prefix}fts_robotside" />
