Commit message: ros_control works well with moveIt! for only one single arm

File: dual_arm_manipulation/dual_arm_robot_description/urdf/dual_arm_robot.urdf.xacro (robot description, xacro)
@@ -1,20 +1,21 @@
-<?xml version="1.0"?> <!--this tag must be in the first line of the xml files-->
-<robot xmlns:xacro="http://www.ros.org/wiki/xacro"
-       name="dual_arm_robot">
-<!-- rosrun xacro xacro.py dual_arm_robot.urdf.xacro >  dual_arm_robot.urdf -->
-  <xacro:property name="pi" value="3.1415926535897931"/>
-  <xacro:arg name="prefix_left" default=""/>
-  <xacro:arg name="prefix_right" default="right_"/>
-  <xacro:arg name="limited" default="true"/>
-  <!-- common stuff -->
-  <xacro:include filename="$(find ur_description)/urdf/common.gazebo.xacro"/>
-  <!-- ur5 -->
-  <xacro:include filename="$(find dual_arm_robot_description)/urdf/ur5.urdf.xacro"/>
-  <!-- ft300 -->
+<?xml version="1.0"?><!--this tag must be in the first line of the xml files-->
+<robot xmlns:xacro="http://wiki.ros.org/xacro" name="dual_arm_robot">
+	<!-- rosrun xacro xacro.py dual_arm_robot.urdf.xacro >  dual_arm_robot.urdf -->
+	<!--Processing Order: Classicly Xacro first loads all includes,
+	    then processes all property and macro definitions and finally instantiates macros and evaluates expressions. -->
+	<!-- common stuff -->
+	<xacro:include filename="$(find ur_description)/urdf/common.gazebo.xacro"/>
+	<!-- ur5 -->
+	<xacro:include filename="$(find dual_arm_robot_description)/urdf/ur5.urdf.xacro"/>
+	<!-- ft300 -->
 	<xacro:include filename="$(find robotiq_ft_sensor)/urdf/robotiq_fts300.urdf.xacro" />
-  <!-- endeffector -->
-  <xacro:include filename="$(find dual_arm_robot_description)/urdf/endeffector.urdf.xacro"/>
-  <xacro:property name="robot_horizontal_stand_width" value="0.5"/>
+	<!-- endeffector -->
+	<xacro:include filename="$(find dual_arm_robot_description)/urdf/endeffector.urdf.xacro"/>
+ 	<xacro:property name="PI" value="3.14159265" />
+	<xacro:property name="robot_horizontal_stand_width" value="0.5"/>
 	<xacro:property name="robot_vertical_stand_height" value="1.2"/>
+	<xacro:arg name="prefix_left" default="left_"/>
+	<xacro:arg name="prefix_right" default="right_"/>
+	<xacro:arg name="limited" default="true"/>
 	<!-- color macros -->
 	<xacro:macro name="material_orange_transparent">
@@ -30,76 +31,41 @@
 	<xacro:material_orange_transparent />
 	<xacro:material_blue_transparent />
-  <!-- end of color macros -->
-  <!-- Stand macros -->
-  <link name="stand1">
-		<visual>
-		<geometry>
-		<cylinder radius="0.08" length="0.8"/>
-		</geometry>
-		<material name="orange_transparent"/>
-		</visual>
-		<collision>
-		<geometry>
-		<cylinder radius="0.08" length="0.8"/>
-		</geometry>
-		<material name="blue_transparent"/>
-		</collision>
-	</link>
-	<link name="stand2">
-		<visual>
-		<geometry>
-		<cylinder radius="0.08" length="${robot_horizontal_stand_width}"/>
-		</geometry>
-		<material name="orange_transparent"/>
-		</visual>
-		<collision>
-		<geometry>
-		<cylinder radius="0.08" length="${robot_horizontal_stand_width}"/>
-		</geometry>
-		<material name="blue_transparent"/>
-		</collision>
-	</link>
-<link name="stand_Base">
-		<visual>
-		<geometry>
-		<cylinder radius="0.5" length="0.7"/>
-		</geometry>
-		<material name="orange_transparent"/>
-		</visual>
-		<collision>
-		<geometry>
-		<cylinder radius="0.5" length="0.7"/>
-		</geometry>
-		<material name="blue_transparent"/>
-		</collision>
-	</link>
-	<link name="table">
-		<visual>
-			<geometry>
-				<box size="1 1.2 0.97" />
-			</geometry>
-			<material name="orange_transparent"/>
-		</visual>
-		<collision>
-			<geometry>
-		<box size="1 1.2 0.92" />
-		</geometry>
-		<material name="blue_transparent"/>
-		</collision>
-	</link>
-  <joint name="table_joint" type="fixed" >
-    <parent link="world" />
-    <child link="table" />
-    <origin xyz="-1 0 0.485" rpy="0 0 0" />
-</joint>
-  <!-- End of stand macros-->
-  <!-- Place the stand in the world -->
-  <link name="world"/>
-    <!-- place world reference -->
-  <joint name="world_to_stand_Base" type="fixed">
+	<!-- end of color macros -->
+	<!-- Stand macros -->
+	<link name="world"/>
+	<link name="stand_Base">
+		<visual>
+			<geometry>
+				<cylinder radius="0.5" length="0.7"/>
+			</geometry>
+			<material name="orange_transparent"/>
+		</visual>
+		<collision>
+			<geometry>
+				<cylinder radius="0.5" length="0.7"/>
+			</geometry>
+			<material name="blue_transparent"/>
+		</collision>
+	</link>
+	<!-- place world reference -->
+	<joint name="world_to_stand_Base" type="fixed">
 		<parent link="world"/>
 		<child link="stand_Base"/>
 		<origin xyz="0 0 0.35" rpy="0 0 0"/>
 	</joint>
+	<link name="stand1">
+		<visual>
+			<geometry>
+				<cylinder radius="0.08" length="0.8"/>
+			</geometry>
+			<material name="orange_transparent"/>
+		</visual>
+		<collision>
+			<geometry>
+				<cylinder radius="0.08" length="0.8"/>
+			</geometry>
+			<material name="blue_transparent"/>
+		</collision>
+	</link>
 	<joint name="Base_to_stand1" type="fixed">
 		<parent link="stand_Base"/>
@@ -107,4 +73,18 @@
 		<origin xyz="0 0 0.6" rpy="0 0 0"/>
 	</joint>
+	<link name="stand2">
+		<visual>
+			<geometry>
+				<cylinder radius="0.08" length="${robot_horizontal_stand_width}"/>
+			</geometry>
+			<material name="orange_transparent"/>
+		</visual>
+		<collision>
+			<geometry>
+				<cylinder radius="0.08" length="${robot_horizontal_stand_width}"/>
+			</geometry>
+			<material name="blue_transparent"/>
+		</collision>
+	</link>
 	<joint name="stand1_to_stand2" type="fixed">
 		<parent link="stand1"/>
@@ -112,56 +92,62 @@
 		<origin xyz="0 0 0.25" rpy="1.57 1.57 0"/>
 	</joint>
-<!-- place a table
-  	<joint name="world_to_table" type="fixed">
-		<parent link="world"/>
-		<child link="table"/>
-		<origin xyz="-1 0 0.5" rpy="0 0 0"/>
-	</joint>
-	-->
-  <!-- place ur5 left arm    -->
-  <xacro:ur5_robot prefix="$(arg prefix_left)" joint_limited="$(arg limited)"/>
-  <joint name="stand2_to_left_arm" type="fixed">
-    <parent link="stand2"/>
-    <child link ="$(arg prefix_left)base_link"/>
-   <origin xyz="0 0 ${(robot_horizontal_stand_width/2)}" rpy="${pi/4.0} 0 0"/>
-  </joint>
-  <!-- place robotiq_fts300 to left arm -->
-  <xacro:robotiq_fts300 prefix="" parent="$(arg prefix_left)ee_link"/>
-  <!-- mount the fts to the robot
-  <joint name="$(arg prefix_left)fts_fix" type="fixed" >
-    <origin xyz="0 0 0" rpy="0 1.57 0"/>
-    <parent link="$(arg prefix_left)ee_link" />
-    <child link="fts_robotside" />
-  </joint>
-	-->
-  <!-- place ur5 endeffector  -->
-  <xacro:endeffector prefix="$(arg prefix_left)"/>
-  <joint name="$(arg prefix_left)ee_mount" type="fixed">
-    <parent link="fts_toolside" />
-    <child link = "$(arg prefix_left)ee_frame" />
-    <origin xyz="0.0 0.0 0.0" rpy="0 0 0 " />
-  </joint>
-<!--
+	<link name="table">
+		<visual>
+			<geometry>
+				<box size="1 1.2 0.97" />
+			</geometry>
+			<material name="orange_transparent"/>
+		</visual>
+		<collision>
+			<geometry>
+				<box size="1 1.2 0.92" />
+			</geometry>
+			<material name="blue_transparent"/>
+		</collision>
+	</link>
+	<joint name="table_joint" type="fixed">
+		<parent link="world" />
+		<child link="table" />
+		<origin xyz="-1 0 0.485" rpy="0 0 0" />
+	</joint>
+	<!-- End of stand macros-->
+	<!-- place ur5 left arm    -->
+	<xacro:ur5_robot prefix="$(arg prefix_left)" joint_limited="$(arg limited)"/>
+	<joint name="stand2_to_left_arm" type="fixed">
+		<parent link="stand2"/>
+		<child link ="$(arg prefix_left)base_link"/>
+		<origin xyz="0 0 ${(robot_horizontal_stand_width/2)}" rpy="${PI/4.0} 0 0"/>
+	</joint>
+	<!-- place robotiq_fts300 to left arm -->
+	<xacro:robotiq_fts300 prefix="" parent="$(arg prefix_left)ee_link"/>
+	<!-- place ur5 endeffector  -->
+	<xacro:endeffector prefix="$(arg prefix_left)"/>
+	<joint name="$(arg prefix_left)ee_mount" type="fixed">
+		<parent link="fts_toolside" />
+		<child link = "$(arg prefix_left)ee_frame" />
+		<origin xyz="0.0 0.0 0.0" rpy="0 0 0 " />
+	</joint>
+	<!--
   <joint name="$(arg prefix_left)ee_mount" type="fixed">
     <parent link="$(arg prefix_left)tool0"/>
     <child link ="$(arg prefix_left)ee_frame"/>
-    <origin xyz="0 0 0" rpy="0 0 ${pi}" />
+    <origin xyz="0 0 0" rpy="0 0 ${PI}" />
   </joint>
 -->
-  <!-- place ur5 right arm  -->
-  <xacro:ur5_robot prefix="$(arg prefix_right)" joint_limited="$(arg limited)"/>
-  <joint name="stand2_to_right_arm" type="fixed">
-    <parent link="stand2"/>
-    <child link ="$(arg prefix_right)base_link"/>
-    <origin xyz="0 0 -${(robot_horizontal_stand_width/2)}" rpy="${pi/4.0} ${pi} 0"/>
-  </joint>
-  <!-- place ur5 right endeffector -->
-  <xacro:endeffector prefix="$(arg prefix_right)"/>
-  <joint name="$(arg prefix_right)ee_mount" type="fixed">
-    <parent link="$(arg prefix_right)ee_link" />
-    <child link = "$(arg prefix_right)ee_frame" />
-    <origin xyz="0.0 0.0 0.0" rpy="${pi/2.0} 0.0 ${pi/2.0}" />
-  </joint>
-  	<link name="wall">
+	<!-- place ur5 right arm  -->
+	<xacro:ur5_robot prefix="$(arg prefix_right)" joint_limited="$(arg limited)"/>
+	<joint name="stand2_to_right_arm" type="fixed">
+		<parent link="stand2"/>
+		<child link ="$(arg prefix_right)base_link"/>
+		<origin xyz="0 0 -${(robot_horizontal_stand_width/2)}" rpy="${PI/4.0} ${PI} 0"/>
+	</joint>
+	<!-- place ur5 right endeffector -->
+	<xacro:endeffector prefix="$(arg prefix_right)"/>
+	<joint name="$(arg prefix_right)ee_mount" type="fixed">
+		<parent link="$(arg prefix_right)ee_link" />
+		<child link = "$(arg prefix_right)ee_frame" />
+		<origin xyz="0.0 0.0 0.0" rpy="${PI/2.0} 0.0 ${PI/2.0}" />
+	</joint>
+	<link name="wall">
 		<visual>
 			<geometry>
@@ -172,15 +158,15 @@
 		<collision>
 			<geometry>
-		<box size="1 1 3" />
-		</geometry>
-		<material name="blue_transparent"/>
-		</collision>
-	</link>
-  <joint name="wall_joint" type="fixed" >
-    <parent link="world" />
-    <child link="wall" />
-    <origin xyz="-1.6 -1.55 1.5" rpy="0 0 0" />
-</joint>
-<link name="wall1">
+				<box size="1 1 3" />
+			</geometry>
+			<material name="blue_transparent"/>
+		</collision>
+	</link>
+	<joint name="wall_joint" type="fixed">
+		<parent link="world" />
+		<child link="wall" />
+		<origin xyz="-1.6 -1.55 1.5" rpy="0 0 0" />
+	</joint>
+	<link name="wall1">
 		<visual>
 			<geometry>
@@ -191,15 +177,15 @@
 		<collision>
 			<geometry>
-		<box size="0.01 2 3" />
-		</geometry>
-		<material name="blue_transparent"/>
-		</collision>
-	</link>
-  <joint name="wall_joint1" type="fixed" >
-    <parent link="world" />
-    <child link="wall1" />
-    <origin xyz="0.5 0 1.5" rpy="0 0 0" />
-</joint>
-<link name="wall2">
+				<box size="0.01 2 3" />
+			</geometry>
+			<material name="blue_transparent"/>
+		</collision>
+	</link>
+	<joint name="wall_joint1" type="fixed">
+		<parent link="world" />
+		<child link="wall1" />
+		<origin xyz="0.5 0 1.5" rpy="0 0 0" />
+	</joint>
+	<link name="wall2">
 		<visual>
 			<geometry>
@@ -210,19 +196,19 @@
 		<collision>
 			<geometry>
-		<box size="2 0.01 3" />
-		</geometry>
-		<material name="blue_transparent"/>
-		</collision>
-	</link>
-  <joint name="wall_joint2" type="fixed" >
-    <parent link="world" />
-    <child link="wall2" />
-    <origin xyz="-1 1.4 1.5" rpy="0 0 0" />
-</joint>
-<!--
+				<box size="2 0.01 3" />
+			</geometry>
+			<material name="blue_transparent"/>
+		</collision>
+	</link>
+	<joint name="wall_joint2" type="fixed">
+		<parent link="world" />
+		<child link="wall2" />
+		<origin xyz="-1 1.4 1.5" rpy="0 0 0" />
+	</joint>
+	<!--
   <joint name="$(arg prefix_right)ee_mount" type="fixed">
     <parent link="$(arg prefix_right)tool0"/>
     <child link ="$(arg prefix_right)ee_frame"/>
-    <origin xyz="0 0 0" rpy="0 0 ${pi}" />
+    <origin xyz="0 0 0" rpy="0 0 ${PI}" />
   </joint>
 -->

File: dual_arm_manipulation/dual_arm_robot_description/urdf/dual_arm_robot_gripper.urdf.xacro (robot description, xacro)
@@ -1,6 +1,6 @@
 <?xml version="1.0"?> <!--this tag must be in the first line of the xml files-->
-<robot xmlns:xacro="http://www.ros.org/wiki/xacro" name="dual_arm_robot">
+<robot xmlns:xacro="http://wiki.ros.org/xacro" name="dual_arm_robot">
 <!-- rosrun xacro xacro.py dual_arm_robot.urdf.xacro >  dual_arm_robot.urdf -->
-  <xacro:property name="pi" value="3.1415926535897931"/>
+  <xacro:property name="PI" value="3.1415926535897931"/>
   <xacro:arg name="prefix_left" default="left_"/>
   <xacro:arg name="prefix_right" default="right_"/>
@@ -185,5 +185,5 @@
     <parent link="stand2"/>
     <child link ="$(arg prefix_left)base_link"/>
-   <origin xyz="0 0 ${(robot_horizontal_stand_width/2)}" rpy="${pi/4.0} 0 0"/>
+   <origin xyz="0 0 ${(robot_horizontal_stand_width/2)}" rpy="${PI/4.0} 0 0"/>
   </joint>
   <!-- place robotiq_fts300 to left arm -->
@@ -225,5 +225,5 @@
     <parent link="flange" />
     <child link = "palm" />
-    <origin xyz="0.0 0 0.06" rpy="${pi/2} 0 0" />
+    <origin xyz="0.0 0 0.06" rpy="${PI/2} 0 0" />
   	</joint>
 <!--
@@ -231,5 +231,5 @@
     <parent link="$(arg prefix_left)tool0"/>
     <child link ="$(arg prefix_left)ee_frame"/>
-    <origin xyz="0 0 0" rpy="0 0 ${pi}" />
+    <origin xyz="0 0 0" rpy="0 0 ${PI}" />
   </joint>
 -->
@@ -239,5 +239,5 @@
     <parent link="stand2"/>
     <child link ="$(arg prefix_right)base_link"/>
-    <origin xyz="0 0 -${(robot_horizontal_stand_width/2)}" rpy="${pi/4.0} ${pi} 0"/>
+    <origin xyz="0 0 -${(robot_horizontal_stand_width/2)}" rpy="${PI/4.0} ${PI} 0"/>
   </joint>
   <!-- place 2 finger gripper on right arm -->
@@ -252,5 +252,5 @@
     <parent link="$(arg prefix_right)tool0"/>
     <child link ="$(arg prefix_right)ee_frame"/>
-    <origin xyz="0 0 0" rpy="0 0 ${pi}" />
+    <origin xyz="0 0 0" rpy="0 0 ${PI}" />
   </joint>
 -->

File: dual_arm_manipulation/dual_arm_robot_description/urdf/endeffector.urdf.xacro (robot description, xacro)
@@ -3,5 +3,5 @@
        xmlns:controller="http://playerstage.sourceforge.net/gazebo/xmlschema/#controller"
        xmlns:interface="http://playerstage.sourceforge.net/gazebo/xmlschema/#interface"
-       xmlns:xacro="http://ros.org/wiki/xacro">
+       xmlns:xacro="http://wiki.ros.org/xacro">
   <xacro:macro name="endeffector" params="prefix">
   <link name="${prefix}ee_frame">

File: dual_arm_manipulation/dual_arm_robot_description/urdf/table.urdf.xacro (robot description, xacro)
@@ -13,13 +13,13 @@
        xmlns:controller="http://playerstage.sourceforge.net/gazebo/xmlschema/#controller"
        xmlns:physics="http://playerstage.sourceforge.net/gazebo/xmlschema/#physics">
-  <property name="table_height" value="0.8" />
-  <property name="table_width" value="1.0" />
-  <property name="table_depth" value="1.0" />
-  <property name="leg_radius" value="0.02" />
-  <property name="table_x" value="0.98" />
-  <property name="table_y" value="0.0" />
-  <property name="table_z" value="0.0" />
-  <property name="table_top_thickness" value="0.05"/>
-  <property name="M_PI" value="3.1415926535897931" />
+  <xacro:property name="table_height" value="0.8" />
+  <xacro:property name="table_width" value="1.0" />
+  <xacro:property name="table_depth" value="1.0" />
+  <xacro:property name="leg_radius" value="0.02" />
+  <xacro:property name="table_x" value="0.98" />
+  <xacro:property name="table_y" value="0.0" />
+  <xacro:property name="table_z" value="0.0" />
+  <xacro:property name="table_top_thickness" value="0.05"/>
+  <xacro:property name="M_PI" value="3.1415926535897931" />
   <xacro:macro name="table">
   <!-- tabletop height is .55+.01+.025=.585 -->

File: dual_arm_manipulation/dual_arm_robot_description/urdf/ur5.urdf.xacro (robot description, xacro)
@@ -1,22 +1,24 @@
 <?xml version="1.0"?>
-<robot xmlns:xacro="http://www.ros.org/wiki/xacro">
+<robot xmlns:xacro="http://wiki.ros.org/xacro">
 <!-- edited by Chunting Jiao-->
   <xacro:include filename="$(find ur_description)/urdf/ur.transmission.xacro" />
   <xacro:include filename="$(find ur_description)/urdf/ur.gazebo.xacro" />
-  <property name="pi" value="3.14159265" />
+<!-- redifining global property: pi
+  <xacro:property name="pi" value="3.14159265" />
+-->
   <!-- Inertia parameters -->
-  <property name="ur5_base_mass" value="4.0" />  <!-- This mass might be incorrect -->
-  <property name="ur5_shoulder_mass" value="3.7000" />
-  <property name="ur5_upper_arm_mass" value="8.3930" />
-  <property name="ur5_forearm_mass" value="2.2750" />
-  <property name="ur5_wrist_1_mass" value="1.2190" />
-  <property name="ur5_wrist_2_mass" value="1.2190" />
-  <property name="ur5_wrist_3_mass" value="0.1879" />
-  <property name="ur5_shoulder_cog" value="0.0 0.00193 -0.02561" />
-  <property name="ur5_upper_arm_cog" value="0.0 -0.024201 0.2125" />
-  <property name="ur5_forearm_cog" value="0.0 0.0265 0.11993" />
-  <property name="ur5_wrist_1_cog" value="0.0 0.110949 0.01634" />
-  <property name="ur5_wrist_2_cog" value="0.0 0.0018 0.11099" />
-  <property name="ur5_wrist_3_cog" value="0.0 0.001159 0.0" />
+  <xacro:property name="ur5_base_mass" value="4.0" />  <!-- This mass might be incorrect -->
+  <xacro:property name="ur5_shoulder_mass" value="3.7000" />
+  <xacro:property name="ur5_upper_arm_mass" value="8.3930" />
+  <xacro:property name="ur5_forearm_mass" value="2.2750" />
+  <xacro:property name="ur5_wrist_1_mass" value="1.2190" />
+  <xacro:property name="ur5_wrist_2_mass" value="1.2190" />
+  <xacro:property name="ur5_wrist_3_mass" value="0.1879" />
+  <xacro:property name="ur5_shoulder_cog" value="0.0 0.00193 -0.02561" />
+  <xacro:property name="ur5_upper_arm_cog" value="0.0 -0.024201 0.2125" />
+  <xacro:property name="ur5_forearm_cog" value="0.0 0.0265 0.11993" />
+  <xacro:property name="ur5_wrist_1_cog" value="0.0 0.110949 0.01634" />
+  <xacro:property name="ur5_wrist_2_cog" value="0.0 0.0018 0.11099" />
+  <xacro:property name="ur5_wrist_3_cog" value="0.0 0.001159 0.0" />
   <!-- Kinematic model -->
   <!-- Properties from urcontrol.conf -->
@@ -31,20 +33,20 @@
     center_of_mass = [ [0, -0.02561, 0.00193], [0.2125, 0, 0.11336], [0.11993, 0.0, 0.0265], [0, -0.0018, 0.01634], [0, 0.0018,0.01634], [0, 0, -0.001159] ]
   -->
-  <property name="ur5_d1" value="0.089159" />
-  <property name="ur5_a2" value="-0.42500" />
-  <property name="ur5_a3" value="-0.39225" />
-  <property name="ur5_d4" value="0.10915" />
-  <property name="ur5_d5" value="0.09465" />
-  <property name="ur5_d6" value="0.0823" />
+  <xacro:property name="ur5_d1" value="0.089159" />
+  <xacro:property name="ur5_a2" value="-0.42500" />
+  <xacro:property name="ur5_a3" value="-0.39225" />
+  <xacro:property name="ur5_d4" value="0.10915" />
+  <xacro:property name="ur5_d5" value="0.09465" />
+  <xacro:property name="ur5_d6" value="0.0823" />
   <!-- Arbitrary offsets for shoulder/elbow joints -->
-  <property name="ur5_shoulder_offset" value="0.13585" />  <!-- measured from model -->
-  <property name="ur5_elbow_offset" value="-0.1197" /> <!-- measured from model -->
+  <xacro:property name="ur5_shoulder_offset" value="0.13585" />  <!-- measured from model -->
+  <xacro:property name="ur5_elbow_offset" value="-0.1197" /> <!-- measured from model -->
   <!-- link lengths used in model -->
-  <property name="ur5_shoulder_height" value="${ur5_d1}" />
-  <property name="ur5_upper_arm_length" value="${-ur5_a2}" />
-  <property name="ur5_forearm_length" value="${-ur5_a3}" />
-  <property name="ur5_wrist_1_length" value="${ur5_d4 - ur5_elbow_offset - ur5_shoulder_offset}" />
-  <property name="ur5_wrist_2_length" value="${ur5_d5}" />
-  <property name="ur5_wrist_3_length" value="${ur5_d6}" />
+  <xacro:property name="ur5_shoulder_height" value="${ur5_d1}" />
+  <xacro:property name="ur5_upper_arm_length" value="${-ur5_a2}" />
+  <xacro:property name="ur5_forearm_length" value="${-ur5_a3}" />
+  <xacro:property name="ur5_wrist_1_length" value="${ur5_d4 - ur5_elbow_offset - ur5_shoulder_offset}" />
+  <xacro:property name="ur5_wrist_2_length" value="${ur5_d5}" />
+  <xacro:property name="ur5_wrist_3_length" value="${ur5_d6}" />
   <!--property name="ur5_shoulder_height" value="0.089159" /-->
   <!--property name="ur5_shoulder_offset" value="0.13585" /-->  <!-- ur5_shoulder_offset - ur5_elbow_offset + ur5_wrist_1_length = 0.10915 -->
@@ -55,13 +57,13 @@
   <!--property name="ur5_wrist_2_length" value="0.09465" /-->   <!-- In CAD this distance is 0.930, but in the spec it is 0.09465 -->
   <!--property name="ur5_wrist_3_length" value="0.0823" /-->
-  <property name="ur5_shoulder_radius" value="0.060" />   <!-- manually measured -->
-  <property name="ur5_upper_arm_radius" value="0.054" />  <!-- manually measured -->
-  <property name="ur5_elbow_radius" value="0.060" />      <!-- manually measured -->
-  <property name="ur5_forearm_radius" value="0.040" />    <!-- manually measured -->
-  <property name="ur5_wrist_radius" value="0.045" />      <!-- manually measured -->
+  <xacro:property name="ur5_shoulder_radius" value="0.060" />   <!-- manually measured -->
+  <xacro:property name="ur5_upper_arm_radius" value="0.054" />  <!-- manually measured -->
+  <xacro:property name="ur5_elbow_radius" value="0.060" />      <!-- manually measured -->
+  <xacro:property name="ur5_forearm_radius" value="0.040" />    <!-- manually measured -->
+  <xacro:property name="ur5_wrist_radius" value="0.045" />      <!-- manually measured -->
   <xacro:macro name="cylinder_inertial" params="radius length mass *origin">
     <inertial>
       <mass value="${mass}" />
-      <insert_block name="origin" />
+      <xacro:insert_block name="origin" />
       <inertia ixx="${0.0833333 * mass * (3 * radius * radius + length * length)}" ixy="0.0" ixz="0.0"
         iyy="${0.0833333 * mass * (3 * radius * radius + length * length)}" iyz="0.0"

File: dual_arm_manipulation/joint_trajectory_admittance_controller/test/rrbot.xacro (robot description, xacro)
@@ -1,5 +1,5 @@
 <?xml version="1.0"?>
 <!-- Revolute-Revolute Manipulator -->
-<robot name="rrbot" xmlns:xacro="http://www.ros.org/wiki/xacro">
+<robot name="rrbot" xmlns:xacro="http://wiki.ros.org/xacro">
   <!-- Constants for robot dimensions -->
   <xacro:property name="PI" value="3.1415926535897931"/>

File: robotiq/robotiq_ft_sensor/urdf/robotiq_fts300.urdf.xacro (robot description, xacro)
@@ -1,4 +1,4 @@
 <?xml version="1.0"?>
-<robot xmlns:xacro="http://www.ros.org/wiki/xacro" name="robotiq_fts300">
+<robot xmlns:xacro="http://wiki.ros.org/xacro" name="robotiq_fts300">
     <xacro:macro name="robotiq_fts300" params="parent prefix">
         <!-- mount the fts to the robot -->
