Commit message: devel-kinetic works
Edit the joint names, group ns, controller names and the relevant parameters

File: dual_arm_manipulation/dual_arm_robot_description/urdf/dual_arm_robot.urdf.xacro (robot description, xacro)
@@ -128,11 +128,4 @@
 		<origin xyz="0.0 0.0 0.0" rpy="0 0 0 " />
 	</joint>
-	<!--
-  <joint name="$(arg prefix_left)ee_mount" type="fixed">
-    <parent link="$(arg prefix_left)tool0"/>
-    <child link ="$(arg prefix_left)ee_frame"/>
-    <origin xyz="0 0 0" rpy="0 0 ${PI}" />
-  </joint>
--->
 	<!-- place ur5 right arm  -->
 	<xacro:ur5_robot prefix="$(arg prefix_right)" joint_limited="$(arg limited)"/>

Commit message: Add FT150 to right arm in urdf and srdf

File: dual_arm_manipulation/dual_arm_robot_description/urdf/dual_arm_robot.urdf.xacro (robot description, xacro)
@@ -10,4 +10,6 @@
 	<!-- ft300 -->
 	<xacro:include filename="$(find robotiq_ft_sensor)/urdf/robotiq_fts300.urdf.xacro" />
+	<!-- ft150 -->
+	<xacro:include filename="$(find robotiq_ft_sensor)/urdf/robotiq_fts150.urdf.xacro" />
 	<!-- endeffector -->
 	<xacro:include filename="$(find dual_arm_robot_description)/urdf/endeffector.urdf.xacro"/>
@@ -120,9 +122,9 @@
 	</joint>
 	<!-- place robotiq_fts300 to left arm -->
-	<xacro:robotiq_fts300 prefix="" parent="$(arg prefix_left)ee_link"/>
+	<xacro:robotiq_fts300 prefix="$(arg prefix_left)" parent="$(arg prefix_left)ee_link"/>
 	<!-- place ur5 endeffector  -->
 	<xacro:endeffector prefix="$(arg prefix_left)"/>
 	<joint name="$(arg prefix_left)ee_mount" type="fixed">
-		<parent link="fts_toolside" />
+		<parent link="$(arg prefix_left)fts_toolside" />
 		<child link = "$(arg prefix_left)ee_frame" />
 		<origin xyz="0.0 0.0 0.0" rpy="0 0 0 " />
@@ -135,10 +137,12 @@
 		<origin xyz="0 0 -${(robot_horizontal_stand_width/2)}" rpy="${PI/4.0} ${PI} 0"/>
 	</joint>
+	<!-- place robotiq_fts150 to right arm -->
+	<xacro:robotiq_fts300 prefix="$(arg prefix_right)" parent="$(arg prefix_right)ee_link"/>
 	<!-- place ur5 right endeffector -->
 	<xacro:endeffector prefix="$(arg prefix_right)"/>
 	<joint name="$(arg prefix_right)ee_mount" type="fixed">
-		<parent link="$(arg prefix_right)ee_link" />
+		<parent link="$(arg prefix_right)fts_toolside" />
 		<child link = "$(arg prefix_right)ee_frame" />
-		<origin xyz="0.0 0.0 0.0" rpy="${PI/2.0} 0.0 ${PI/2.0}" />
+		<origin xyz="0.0 0.0 0.0" rpy="0 0.0 0" />
 	</joint>
 	<link name="wall">

File: robotiq/robotiq_ft_sensor/urdf/robotiq_fts150.urdf.xacro (robot description, xacro)
@@ -1,9 +1,9 @@
 <?xml version="1.0"?>
-<robot xmlns:xacro="http://ros.org/wiki/xacro" name="robotiq_fts150">
+<robot xmlns:xacro="http://wiki.ros.org/xacro" name="robotiq_fts150">
     <xacro:macro name="robotiq_fts150" params="parent prefix *origin">
         <!-- mount the fts to the robot -->
         <joint name="${prefix}fts_fix" type="fixed" >
             <!--In most cases origin would be flange adapter plate: <origin xyz="0 0 0.009" rpy="0 0 0"/> /-->
-            <insert_block name="origin" />
+            <origin xyz="0 0 0" rpy="0 1.57 0"/>
             <parent link="${parent}" />
             <child link="${prefix}fts_robotside" />

File: robotiq/robotiq_ft_sensor/urdf/robotiq_fts300.urdf.xacro (robot description, xacro)
@@ -4,5 +4,5 @@
         <!-- mount the fts to the robot -->
         <joint name="${prefix}fts_fix" type="fixed" >
-            <origin xyz="0 0 -0.009" rpy="0 1.57 0"/>
+            <origin xyz="0 0 -0" rpy="0 1.57 0"/>
             <parent link="${parent}" />
             <child link="${prefix}fts_robotside" />

File: universal_robot/ur_description/urdf/ur5_robot.urdf.xacro (robot description, xacro)
@@ -23,5 +23,5 @@
   <xacro:endeffector prefix="$(arg prefix)"/>
   <joint name="$(arg prefix)ee_mount" type="fixed">
-		<parent link="fts_toolside" />
+		<parent link="$(arg prefix)fts_toolside" />
 		<child link = "$(arg prefix)ee_frame" />
 		<origin xyz="0.0 0.0 0.0" rpy="0 0 0 " />

Commit message: Add the serial id for ft sensor

File: dual_arm_manipulation/dual_arm_robot_description/urdf/dual_arm_robot.urdf.xacro (robot description, xacro)
@@ -97,11 +97,11 @@
 		<visual>
 			<geometry>
-				<box size="1 1.2 0.97" />
-			</geometry>
-			<material name="orange_transparent"/>
-		</visual>
-		<collision>
-			<geometry>
-				<box size="1 1.2 0.92" />
+				<box size="1 1.2 0.90" />
+			</geometry>
+			<material name="orange_transparent"/>
+		</visual>
+		<collision>
+			<geometry>
+				<box size="1 1.2 0.90" />
 			</geometry>
 			<material name="blue_transparent"/>
@@ -111,5 +111,5 @@
 		<parent link="world" />
 		<child link="table" />
-		<origin xyz="-1 0 0.485" rpy="0 0 0" />
+		<origin xyz="-1 0 0.45" rpy="0 0 0" />
 	</joint>
 	<!-- End of stand macros-->

Commit message: Start to merge cartesian control to dual_arm_control

File: dual_arm_manipulation/dual_arm_robot_description/urdf/dual_arm_robot.urdf.xacro (robot description, xacro)
@@ -19,5 +19,5 @@
 	<xacro:arg name="prefix_left" default="left_"/>
 	<xacro:arg name="prefix_right" default="right_"/>
-	<xacro:arg name="limited" default="true"/>
+	<xacro:arg name="limited" default="false"/>
 	<!-- color macros -->
 	<xacro:macro name="material_orange_transparent">

File: dual_arm_manipulation/dual_arm_robot_description/urdf/ur5.urdf.xacro (robot description, xacro)
@@ -127,5 +127,5 @@
       <axis xyz="0 1 0" />
       <xacro:unless value="${joint_limited}">
-        <limit lower="${-pi}" upper="${pi}" effort="150.0" velocity="2"/>
+        <limit lower="${-2*pi}" upper="${2*pi}" effort="150.0" velocity="2"/>
       </xacro:unless>
       <xacro:if value="${joint_limited}">
@@ -279,5 +279,4 @@
       <parent link="${prefix}wrist_3_link" />
       <child link = "${prefix}ee_link" />
-      <!--origin xyz="0.0 ${ur5_wrist_3_length} 0.0" rpy="${pi/2} ${pi} ${-pi}" /-->
       <origin xyz="0.0 ${ur5_wrist_3_length} 0.0" rpy="0.0 0.0 ${pi/2.0}" />
     </joint>

Commit message: Pure position control

File: dual_arm_manipulation/dual_arm_robot_description/urdf/dual_arm_robot.urdf.xacro (robot description, xacro)
@@ -97,11 +97,11 @@
 		<visual>
 			<geometry>
-				<box size="1 1.2 0.90" />
-			</geometry>
-			<material name="orange_transparent"/>
-		</visual>
-		<collision>
-			<geometry>
-				<box size="1 1.2 0.90" />
+				<box size="1.2 0.5 0.90" />
+			</geometry>
+			<material name="orange_transparent"/>
+		</visual>
+		<collision>
+			<geometry>
+				<box size="1.2 0.5 0.90" />
 			</geometry>
 			<material name="blue_transparent"/>
@@ -111,5 +111,5 @@
 		<parent link="world" />
 		<child link="table" />
-		<origin xyz="-1 0 0.45" rpy="0 0 0" />
+		<origin xyz="-1.2 0 0.45" rpy="0 0 0" />
 	</joint>
 	<!-- End of stand macros-->

Commit message: Change the connection in ur5.urdf.xacro.
To make the transform from the tip to root be coincident with that in teachPad.
The ${prefix}base_link is replaced by ${prefix}base and ${prefix}ee_link is replaced by ${prefix}tool0. Also connect ${prefix}shoulder_link to ${prefix}base, the rpy changed accordingly. 
2. Since the tip link is changed, the the connection between ft sensor and tip link is also changed.

File: dual_arm_manipulation/dual_arm_robot_description/urdf/dual_arm_robot.urdf.xacro (robot description, xacro)
@@ -122,5 +122,5 @@
 	</joint>
 	<!-- place robotiq_fts300 to left arm -->
-	<xacro:robotiq_fts300 prefix="$(arg prefix_left)" parent="$(arg prefix_left)ee_link"/>
+	<xacro:robotiq_fts300 prefix="$(arg prefix_left)" parent="$(arg prefix_left)tool0"/>
 	<!-- place ur5 endeffector  -->
 	<xacro:endeffector prefix="$(arg prefix_left)"/>
@@ -138,5 +138,5 @@
 	</joint>
 	<!-- place robotiq_fts150 to right arm -->
-	<xacro:robotiq_fts300 prefix="$(arg prefix_right)" parent="$(arg prefix_right)ee_link"/>
+	<xacro:robotiq_fts300 prefix="$(arg prefix_right)" parent="$(arg prefix_right)tool0"/>
 	<!-- place ur5 right endeffector -->
 	<xacro:endeffector prefix="$(arg prefix_right)"/>

File: dual_arm_manipulation/dual_arm_robot_description/urdf/ur5.urdf.xacro (robot description, xacro)
@@ -90,8 +90,12 @@
       </xacro:cylinder_inertial>
     </link>
+    <!--This connection is different from the original one (ur_description).
+        The parent link is changed from ${prefix}base_link to ${prefix}base,
+        then the transform from the base to tool0 is coincident with teachPad.
+        The joint rpy is adjusted to rpy="0 0 ${pi}", if connected to ${prefix}base_link, it should be rpy="0 0 0" -->
     <joint name="${prefix}shoulder_pan_joint" type="revolute">
-      <parent link="${prefix}base_link" />
+      <parent link="${prefix}base" />
       <child link = "${prefix}shoulder_link" />
-      <origin xyz="0.0 0.0 ${ur5_shoulder_height}" rpy="0.0 0.0 0.0" />
+      <origin xyz="0.0 0.0 ${ur5_shoulder_height}" rpy="0 0 ${pi}" />
       <axis xyz="0 0 1" />
       <xacro:unless value="${joint_limited}">

File: robotiq/robotiq_ft_sensor/urdf/robotiq_fts300.urdf.xacro (robot description, xacro)
@@ -4,5 +4,5 @@
         <!-- mount the fts to the robot -->
         <joint name="${prefix}fts_fix" type="fixed" >
-            <origin xyz="0 0 -0" rpy="0 1.57 0"/>
+            <origin xyz="0 0 -0" rpy="0 0 0"/>
             <parent link="${parent}" />
             <child link="${prefix}fts_robotside" />

Commit message: Draw a circle with computeCartesianPath

File: dual_arm_manipulation/dual_arm_robot_description/urdf/dual_arm_robot.urdf.xacro (robot description, xacro)
@@ -97,11 +97,11 @@
 		<visual>
 			<geometry>
-				<box size="1.2 0.5 0.90" />
-			</geometry>
-			<material name="orange_transparent"/>
-		</visual>
-		<collision>
-			<geometry>
-				<box size="1.2 0.5 0.90" />
+				<box size="1.2 0.8 0.90" />
+			</geometry>
+			<material name="orange_transparent"/>
+		</visual>
+		<collision>
+			<geometry>
+				<box size="1.2 0.8 0.90" />
 			</geometry>
 			<material name="blue_transparent"/>
